File: PCB1 PANEL_IN SPV1040 BUCK5 BUCK33 OCPC/_autosave-SPV1040_1.kicad_sch (KiCad schematic)
At the start: 14 parts, among them J2 SOLAR, U2 SPV1040TTR

Commit message: 2
Connections:
- no-connect marks 4 -> 0
Changed lines of the file:
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@@
 		(color 0 0 0 0)
-	)
-	(no_connect
-		(at 91.44 148.59)
-	)
-	(no_connect
-		(at 102.87 148.59)
-	)
-	(no_connect
-		(at 99.06 148.59)
-	)
-	(no_connect
-		(at 86.36 148.59)
 	)
 	(wire
