File: PCB1 PANEL_IN SPV1040 BUCK5 BUCK33 OCPC/USB_CHARGER.kicad_sch (KiCad schematic)
At the start: 16 parts, among them J1 Conn_01x06, U1 BQ25883RGER

Commit message: 2
Other:
- company: (none) -> TEAM ANANT
Changed lines of the file:
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@@
 	(generator_version "8.0")
 	(paper "A4")
+	(title_block
+		(company "TEAM ANANT")
+		(comment 1 "BITS PILANI")
+	)
 	(junction
 		(at 133.35 124.46)

Commit message: EDITS NTH
Parts:
- added J10: USB_C_Receptacle_USB2.0_16P, Connector_USB:USB_C_Receptacle_G-Switch_GT-USB-7010ASV, symbol Connector:USB_C_Receptacle_USB2.0_16P
Connections:
- net GND: now also C1.1, C3.1, C7.1, J1.6 (Pin_6), U1.19 (GND_1), U1.20 (GND_2), U1.25 (EP), J10.A1 (GND), J10.A12 (GND), J10.B1 (GND), J10.B12 (GND), J10.S1 (SHIELD)
- net GNDREF: no longer C1.1, C3.1, C7.1, J1.6 (Pin_6), U1.19 (GND_1), U1.20 (GND_2), U1.25 (EP)
- net USB_D+: now also J10.A6 (D+), J10.B6 (D+)
- net USB_D-: now also J10.A7 (D-), J10.B7 (D-)
- net VBUS_IN: now also J10.A4 (VBUS), J10.A9 (VBUS), J10.B4 (VBUS), J10.B9 (VBUS)
- no-connect marks 4 -> 8
Other:
- note added: "GARBAGE PART REMOVE AND ADD TO THE BUS"

Commit message: .
Parts:
- C1: JLC Part  (none) -> C1592
- C2: JLC Part  (none) -> C19666
- C3, C7: JLC Part  (none) -> C96446
- C4: JLC Part  (none) -> C113811
- C5, C6: JLC Part  (none) -> C6119868
- D1: JLC Part  (none) -> C2994781
- J10: JLC Part  (none) -> C2988369
- L1: JLC Part  (none) -> C7038984
- R2: JLC Part  (none) -> C140082
- R3: JLC Part  (none) -> C321843
- R4, R6: JLC Part  (none) -> C115324
- R5: JLC Part  (none) -> C100959
- U1: JLC Part  (none) -> C544362
