File: PCB1 PANEL_IN SPV1040 BUCK5 BUCK33 OCPC/SPV1040_1.kicad_sch (KiCad schematic)
At the start: 14 parts, among them J2 SOLAR, U2 SPV1040TTR

Commit message: Relabeling according to standards
Parts:
- D1401: renamed from CR4; footprint CR_F5.0A-TR_STM -> (none)
- renumbered C8 to C1401, C_IN1 to C1402, C_out1 to C1403, C_out2 to C1404, C9 to C1405, D6 to D1402, J2 to J1401, L2 to L1401, R7 to R1401, R10 to R1402, R9 to R1403, SUPER_CAP1 to SUPER_CAP1401, U2 to U1401
Changed lines of the file:
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@@
 		(on_board yes)
 		(dnp no)
-		(property "Reference" "SUPER_CAP1"
+		(property "Reference" "SUPER_CAP1401"
 			(at 255.27 72.39 90)
 			(effects
@@
 			(project "PCB1 PANEL_IN SPV1040 BUCK5 BUCK33 OCPC"
 				(path "/494c9d9f-6b33-4248-a813-27ffaaa929bd/e53a10ab-2cc0-41d1-82dc-2525f18f01bb"
-					(reference "SUPER_CAP1")
+					(reference "SUPER_CAP1401")
 					(unit 1)
 				)
@@
 		(dnp no)
 		(fields_autoplaced yes)
-		(property "Reference" "C_out1"
+		(property "Reference" "C1403"
 			(at 92.71 101.5999 0)
 			(effects
@@
 			(project "PCB1 PANEL_IN SPV1040 BUCK5 BUCK33 OCPC"
 				(path "/494c9d9f-6b33-4248-a813-27ffaaa929bd/e53a10ab-2cc0-41d1-82dc-2525f18f01bb"
-					(reference "C_out1")
+					(reference "C1403")
 					(unit 1)
 				)
@@
 		(dnp no)
 		(fields_autoplaced yes)
-		(property "Reference" "C8"
+		(property "Reference" "C1401"
 			(at 68.58 38.0999 0)
 			(effects
@@
 			(project "PCB1 PANEL_IN SPV1040 BUCK5 BUCK33 OCPC"
 				(path "/494c9d9f-6b33-4248-a813-27ffaaa929bd/e53a10ab-2cc0-41d1-82dc-2525f18f01bb"
-					(reference "C8")
+					(reference "C1401")
 					(unit 1)
 				)
@@
 		(on_board yes)
 		(dnp no)
-		(property "Reference" "R9"
+		(property "Reference" "R1403"
 			(at 167.64 76.2 90)
 			(effects
@@
 			(project "PCB1 PANEL_IN SPV1040 BUCK5 BUCK33 OCPC"
 				(path "/494c9d9f-6b33-4248-a813-27ffaaa929bd/e53a10ab-2cc0-41d1-82dc-2525f18f01bb"
-					(reference "R9")
+					(reference "R1403")
 					(unit 1)
 				)
@@
 		(dnp no)
 		(fields_autoplaced yes)
-		(property "Reference" "C9"
+		(property "Reference" "C1405"
 			(at 129.54 86.3599 0)
 			(effects
@@
 			(project "PCB1 PANEL_IN SPV1040 BUCK5 BUCK33 OCPC"
 				(path "/494c9d9f-6b33-4248-a813-27ffaaa929bd/e53a10ab-2cc0-41d1-82dc-2525f18f01bb"
-					(reference "C9")
+					(reference "C1405")
 					(unit 1)
 				)
@@
 		(on_board yes)
 		(dnp no)
-		(property "Reference" "R10"
+		(property "Reference" "R1402"
 			(at 167.64 91.44 90)
 			(effects
@@
 			(project "PCB1 PANEL_IN SPV1040 BUCK5 BUCK33 OCPC"
 				(path "/494c9d9f-6b33-4248-a813-27ffaaa929bd/e53a10ab-2cc0-41d1-82dc-2525f18f01bb"
-					(reference "R10")
+					(reference "R1402")
 					(unit 1)
 				)
@@
 		(dnp no)
 		(fields_autoplaced yes)
-		(property "Reference" "C_out2"
+		(property "Reference" "C1404"
 			(at 177.8 86.3599 0)
 			(effects
@@
 			(project "PCB1 PANEL_IN SPV1040 BUCK5 BUCK33 OCPC"
 				(path "/494c9d9f-6b33-4248-a813-27ffaaa929bd/e53a10ab-2cc0-41d1-82dc-2525f18f01bb"
-					(reference "C_out2")
+					(reference "C1404")
 					(unit 1)
 				)
@@
 		(on_board yes)
 		(dnp no)
-		(property "Reference" "C_IN1"
+		(property "Reference" "C1402"
 			(at 137.16 34.29 90)
 			(effects
@@
 			(project "PCB1 PANEL_IN SPV1040 BUCK5 BUCK33 OCPC"
 				(path "/494c9d9f-6b33-4248-a813-27ffaaa929bd/e53a10ab-2cc0-41d1-82dc-2525f18f01bb"
-					(reference "C_IN1")
+					(reference "C1402")
 					(unit 1)
 				)
@@
 		(on_board yes)
 		(dnp no)
-		(property "Reference" "D6"
-			(at 96.2026 151.13 0)
+		(property "Reference" "D1402"
+			(at 102.362 151.13 0)
 			(effects
 				(font
@@
 			(project "PCB1 PANEL_IN SPV1040 BUCK5 BUCK33 OCPC"
 				(path "/494c9d9f-6b33-4248-a813-27ffaaa929bd/e53a10ab-2cc0-41d1-82dc-2525f18f01bb"
-					(reference "D6")
+					(reference "D1402")
 					(unit 1)
 				)
@@
 		(dnp no)
 		(fields_autoplaced yes)
-		(property "Reference" "U2"
+		(property "Reference" "U1401"
 			(at 95.25 54.61 0)
 			(effects
@@
 			(project "PCB1 PANEL_IN SPV1040 BUCK5 BUCK33 OCPC"
 				(path "/494c9d9f-6b33-4248-a813-27ffaaa929bd/e53a10ab-2cc0-41d1-82dc-2525f18f01bb"
-					(reference "U2")
+					(reference "U1401")
 					(unit 1)
 				)
@@
 		(dnp no)
 		(fields_autoplaced yes)
-		(property "Reference" "L2"
+		(property "Reference" "L1401"
 			(at 121.92 33.02 90)
 			(effects
@@
 			(project "PCB1 PANEL_IN SPV1040 BUCK5 BUCK33 OCPC"
 				(path "/494c9d9f-6b33-4248-a813-27ffaaa929bd/e53a10ab-2cc0-41d1-82dc-2525f18f01bb"
-					(reference "L2")
+					(reference "L1401")
 					(unit 1)
 				)
@@
 		(dnp no)
 		(fields_autoplaced yes)
-		(property "Reference" "R7"
+		(property "Reference" "R1401"
 			(at 128.27 43.1799 0)
 			(effects
@@
 			(project "PCB1 PANEL_IN SPV1040 BUCK5 BUCK33 OCPC"
 				(path "/494c9d9f-6b33-4248-a813-27ffaaa929bd/e53a10ab-2cc0-41d1-82dc-2525f18f01bb"
-					(reference "R7")
+					(reference "R1401")
 					(unit 1)
 				)
@@
 		(dnp no)
 		(fields_autoplaced yes)
-		(property "Reference" "J2"
+		(property "Reference" "J1401"
 			(at 185.42 36.8299 90)
 			(effects
@@
 			(project "PCB1 PANEL_IN SPV1040 BUCK5 BUCK33 OCPC"
 				(path "/494c9d9f-6b33-4248-a813-27ffaaa929bd/e53a10ab-2cc0-41d1-82dc-2525f18f01bb"
-					(reference "J2")
+					(reference "J1401")
 					(unit 1)
 				)
@@
 		(dnp no)
 		(fields_autoplaced yes)
-		(property "Reference" "CR4"
+		(property "Reference" "D1401"
 			(at 102.87 88.9 0)
 			(effects
@@
 			)
 		)
-		(property "Footprint" "CR_F5.0A-TR_STM"
+		(property "Footprint" ""
 			(at 97.79 95.25 0)
 			(effects
@@
 			(project "PCB1 PANEL_IN SPV1040 BUCK5 BUCK33 OCPC"
 				(path "/494c9d9f-6b33-4248-a813-27ffaaa929bd/e53a10ab-2cc0-41d1-82dc-2525f18f01bb"
-					(reference "CR4")
-					(unit 1)
-				)
+					(reference "D1401")
+					(unit 1)
+				)
