File: PCB1 PANEL_IN SPV1040 BUCK5 BUCK33 OCPC/BUCK3_3.kicad_sch (KiCad schematic)
At the start: 19 parts, among them U8 LM21305SQ/NOPB

Commit message: Relabeling according to standards
Parts:
- removed C18: 2u2, Capacitor_Tantalum_SMD:CP_EIA-7343-43_Kemet-X_Pad2.25x2.55mm_HandSolder, symbol Device:C_Small
- removed C19, C20, C21, C22, C23, C24, C25, C26: 2u2, Capacitor_SMD:C_0603_1608Metric_Pad1.08x0.95mm_HandSolder, symbol Device:C_Small
- removed L8: L, Inductor_SMD:L_6.3x6.3_H3, symbol Device:L
- removed R23, R24, R25, R26, R27, R28, R29, R30: 1k, Resistor_SMD:R_0603_1608Metric_Pad0.98x0.95mm_HandSolder, symbol Device:R_Small
- removed U8: LM21305SQ/NOPB, footprintLM21305:LM21305SQ&slash_NOPB, symbol 2023-03-29_16-01-02:LM21305SQ/NOPB
