File: PCB1 PANEL_IN SPV1040 BUCK5 BUCK33 OCPC/DATA_BUS.kicad_sch (KiCad schematic)
At the start: 45 parts, among them Q1 BSS138DWQ-7, Q2 BSS138DWQ-7, Q3 MBT2222ADW1T1, Q4 MBT2222ADW1T1, Q5 BSS138DWQ-7, Q6 BSS138DWQ-7, Q7 MBT2222ADW1T1, Q8 MBT2222ADW1T1, Q9 MMDT2907, U23 Payload

Commit message: Relabeling according to standards
Parts:
- renumbered C53 to C901, C55 to C902, C54 to C903, C56 to C904, JP1 to JP901, JP2 to JP902, JP3 to JP903, JP4 to JP904, JP5 to JP905, JP6 to JP906, JP7 to JP907, Q1 to M901, Q5 to M902, Q2 to M903, Q2 to M904, R66 to R901, R68 to R902, R64 to R903, R62 to R904, R69 to R905, R76 to R906, R78 to R907, R74 to R908, R72 to R909, R79 to R910, R67 to R911, R70 to R912, R65 to R913, R63 to R914, R71 to R915, R77 to R916, R80 to R917, R75 to R918, R73 to R919, R81 to R920, R83 to R921, R82 to R922, R84 to R923, R85 to R924, Q3 to T901, Q7 to T902, Q4 to T903, Q8 to T904, Q9 to T905, U23 to U901
