File: PCB1 PANEL_IN SPV1040 BUCK5 BUCK33 OCPC/DATA_BUS.kicad_sch (KiCad schematic)
At the start: 45 parts, among them Q1 BSS138DWQ-7, Q2 BSS138DWQ-7, Q3 MBT2222ADW1T1, Q4 MBT2222ADW1T1, Q5 BSS138DWQ-7, Q6 BSS138DWQ-7, Q7 MBT2222ADW1T1, Q8 MBT2222ADW1T1, Q9 MMDT2907, U23 Payload

Commit message: VCOMMIT
EDITS N+I
Parts:
- removed C53, C54, C55, C56: 10nF, Capacitor_SMD:C_0603_1608Metric, symbol Device:C
- removed JP1, JP2, JP3, JP4: SolderJumper_2_Open, Jumper:SolderJumper-2_P1.3mm_Open_RoundedPad1.0x1.5mm, symbol Jumper:SolderJumper_2_Open
- removed Q1, Q2, Q5, Q6: BSS138DWQ-7, mainboard:BSS138DWQ-7, symbol mainboard:BSS138DWQ-7
- removed Q3, Q4, Q7, Q8: MBT2222ADW1T1, Package_TO_SOT_SMD:SOT-363_SC-70-6, symbol Transistor_BJT:MBT2222ADW1T1
- removed Q9: MMDT2907, Package_TO_SOT_SMD:SOT-363_SC-70-6, symbol mainboard:MMDT2907
- removed R62, R63, R72, R73: 100K, Resistor_SMD:R_0603_1608Metric, symbol Device:R_US
- removed R64, R65, R74, R75: 680, Resistor_SMD:R_0603_1608Metric, symbol Device:R_US
- removed R66, R67, R68, R70, R76, R77, R78, R80: 10K, Resistor_SMD:R_0603_1608Metric, symbol Device:R_US
- removed R69, R71, R79, R81: 200K, Resistor_SMD:R_0603_1608Metric, symbol Device:R_US
- removed R82: 0, Resistor_SMD:R_0603_1608Metric, symbol Device:R_US
- removed R83: 4.7K, Resistor_SMD:R_0603_1608Metric, symbol Device:R_US
- removed R84, R85: 1K, Resistor_SMD:R_0603_1608Metric, symbol Device:R_US
- removed U23: Payload, symbol PC104:Payload
Other:
- added sheet I2C_PROTEC (I2C_PROTEC.kicad_sch)
- added sheet PC104 (PC104.kicad_sch)
- added sheet SPI_PROTEC (SPI_PROTEC.kicad_sch)
- note removed: "Bus Protection - Bypass Jumpers"
- note removed: "REPLACE THINKING ABOUT INTERFERENCE AND EMI SHIT"
- note removed: "SPI Bus Protection - CHECK BEFORE IMPLEMENTATION"
