File: PCB1 PANEL_IN SPV1040 BUCK5 BUCK33 OCPC/INA219.kicad_sch (KiCad schematic)
At the start: 17 parts, among them U10 INA219BxDCN, U11 INA219BxDCN, U12 INA219BxDCN, U13 INA219BxDCN, U9 INA219BxDCN

Commit message: Update INA219.kicad_sch
Connections:
- net 3V3_BUS renamed 3.3V_ADCS
- net 5V_BUS renamed 5V_ADCSC
- net OBC_5V renamed 5V_OBC
- net PAY_5V renamed 5V_PAYLOAD
- net TTC_3V3 renamed 3.3v_TTC
Other:
- note added: "I2C BUS ADDR: 0x44(1000100)"
- note added: "I2C BUS ADDR: 0x45(1000101)"
- note added: "I2C BUS ADDR: 0x4F(1001111)"
- note added: "I2C BUS ADDR:0x40(1000000)"
- note added: "I2C BUS ADDR:0x4A (1001010)"
- note removed: "I2C BUS ADDR:"
Changed lines of the file:
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@@
 	(wire
 		(pts
-			(xy 241.3 104.14) (xy 241.3 118.11)
-		)
-		(stroke
-			(width 0)
-			(type default)
-		)
-	)
-	(wire
-		(pts
 			(xy 57.15 113.03) (xy 62.23 113.03)
 		)
@@
 	(wire
 		(pts
+			(xy 223.52 91.44) (xy 223.52 114.3)
+		)
+		(stroke
+			(width 0)
+			(type default)
+		)
+	)
+	(wire
+		(pts
 			(xy 130.81 30.48) (xy 130.81 40.64)
 		)
@@
 	(wire
 		(pts
+			(xy 241.3 92.71) (xy 241.3 118.11)
+		)
+		(stroke
+			(width 0)
+			(type default)
+		)
+	)
+	(wire
+		(pts
 			(xy 129.54 95.25) (xy 133.35 95.25)
 		)
@@
 	(wire
 		(pts
-			(xy 223.52 101.6) (xy 223.52 114.3)
-		)
-		(stroke
-			(width 0)
-			(type default)
-		)
-	)
-	(wire
-		(pts
 			(xy 204.47 46.99) (xy 201.93 46.99)
 		)
@@
 	)
 	(rectangle
-		(start 205.74 95.25)
-		(end 260.35 142.24)
+		(start 204.47 88.9)
+		(end 259.08 135.89)
 		(stroke
 			(width 0)
@@
 		)
 	)
-	(text "I2C BUS ADDR:"
+	(text "I2C BUS ADDR: 0x4F(1001111)"
 		(exclude_from_sim no)
-		(at 122.174 71.628 0)
+		(at 135.89 71.12 0)
 		(effects
 			(font
@@
 		)
 	)
-	(text "I2C BUS ADDR:"
+	(text "I2C BUS ADDR:0x40(1000000)\n"
 		(exclude_from_sim no)
-		(at 32.004 71.882 0)
+		(at 44.45 72.39 0)
 		(effects
 			(font
@@
 		)
 	)
-	(text "I2C BUS ADDR:"
+	(text "I2C BUS ADDR: 0x44(1000100)\n"
 		(exclude_from_sim no)
-		(at 116.586 137.668 0)
+		(at 129.54 137.16 0)
 		(effects
 			(font
@@
 		)
 	)
-	(text "I2C BUS ADDR:"
+	(text "I2C BUS ADDR: 0x45(1000101)"
 		(exclude_from_sim no)
-		(at 32.004 135.89 0)
+		(at 40.64 135.89 0)
 		(effects
 			(font
@@
 		)
 	)
-	(text "I2C BUS ADDR:"
+	(text "I2C BUS ADDR:0x4A (1001010)"
 		(exclude_from_sim no)
-		(at 199.898 72.39 0)
+		(at 218.44 72.39 0)
 		(effects
 			(font
@@
 		)
 	)
-	(label "TTC_3V3"
+	(label "3.3v_TTC"
 		(at 160.02 46.99 0)
 		(fields_autoplaced yes)
@@
 		)
 	)
-	(label "5V_BUS"
+	(label "5V_ADCSC"
 		(at 71.12 113.03 0)
 		(fields_autoplaced yes)
@@
 		)
 	)
-	(label "OBC_5V"
+	(label "5V_OBC"
 		(at 71.12 46.99 0)
 		(fields_autoplaced yes)
@@
 		)
 	)
-	(label "3V3_BUS"
+	(label "3.3V_ADCS"
 		(at 158.75 111.76 0)
 		(fields_autoplaced yes)
@@
 		)
 	)
-	(label "PAY_5V"
+	(label "5V_PAYLOAD"
 		(at 243.84 48.26 0)
 		(fields_autoplaced yes)
@@
 		)
 	)
-	(label "SDA"
-		(at 223.52 107.95 90)
+	(label "I2C_5V_PROTEC_SDA"
+		(at 223.52 111.76 90)
 		(fields_autoplaced yes)
 		(effects
@@
 		)
 	)
-	(label "SCL"
-		(at 241.3 109.22 90)
+	(label "I2C_5V_PROTEC_SCL"
+		(at 241.3 113.03 90)
 		(fields_autoplaced yes)
 		(effects
@@
 		(dnp no)
 		(property "Reference" "R37"
-			(at 219.71 107.95 90)
+			(at 215.9 110.49 90)
 			(effects
 				(font
@@
 		)
 		(property "Value" "10k"
-			(at 219.71 110.49 90)
+			(at 219.71 114.3 90)
 			(effects
 				(font
@@
 		)
 	)
+	(sheet_instances
+		(path "/"
+			(page "1")
+		)
+	)

Commit message: .
Parts:
- C?: renamed from C38; JLC PART NUMBER (none) -> C338036
- C?: renamed from C40; JLC PART NUMBER (none) -> C338036
- C?: renamed from C36; JLC PART NUMBER (none) -> C338036
- C?: renamed from C37; JLC PART NUMBER (none) -> C338036
- C?: renamed from C39; JLC PART NUMBER (none) -> C338036
- R?: renamed from R46; JLC PART NUMBER (none) -> C2907569
- R?: renamed from R38; JLC PART NUMBER (none) -> C328655
- R?: renamed from R37; JLC PART NUMBER (none) -> C328655
- R?: renamed from R51; JLC PART NUMBER (none) -> C2907569
- R?: renamed from R61; JLC PART NUMBER (none) -> C2907569
- R?: renamed from R41; JLC PART NUMBER (none) -> C2907569
- R?: renamed from R56; JLC PART NUMBER (none) -> C2907569
- U?: renamed from U11; JLC PART NUMBER (none) -> C2653868
- U?: renamed from U9; JLC PART NUMBER (none) -> C2653868
- U?: renamed from U12; JLC PART NUMBER (none) -> C2653868
- U?: renamed from U10; JLC PART NUMBER (none) -> C2653868
- U?: renamed from U13; JLC PART NUMBER (none) -> C2653868
