File: PCB1 PANEL_IN SPV1040 BUCK5 BUCK33 OCPC/INA219.kicad_sch (KiCad schematic)
At the start: 17 parts, among them U10 INA219BxDCN, U11 INA219BxDCN, U12 INA219BxDCN, U13 INA219BxDCN, U9 INA219BxDCN

Commit message: VCOMMIT
EDITS N+I
Parts:
- removed C36, C37, C38, C39, C40: 100n, Capacitor_SMD:C_0603_1608Metric, symbol Device:C
- removed R37, R38: 10k, Resistor_SMD:R_0603_1608Metric, symbol Device:R
- removed R41, R46, R51, R56, R61: R100, Resistor_SMD:R_2512_6332Metric, symbol Device:R
- removed U10, U11, U12, U13, U9: INA219BxDCN, Package_TO_SOT_SMD:SOT-23-8, symbol Sensor_Energy:INA219BxDCN
Other:
- note removed: "I2C BUS ADDR: 0x44(1000100)"
- note removed: "I2C BUS ADDR: 0x45(1000101)"
- note removed: "I2C BUS ADDR: 0x4F(1001111)"
- note removed: "I2C BUS ADDR:0x40(1000000)"
- note removed: "I2C BUS ADDR:0x4A (1001010)"
