File: PCB1 PANEL_IN SPV1040 BUCK5 BUCK33 OCPC/OCPC.kicad_sch (KiCad schematic)
At the start: 35 parts, among them J11 Conn_01x02_Pin, J12 Conn_01x02_Pin, J13 OCPC_EN, J14 OCPC_EN, J15 OCPC_EN, J16 OCPC_EN, J17 OCPC_EN, J7 Conn_01x02_Pin, J8 Conn_01x02_Pin, J9 Conn_01x02_Pin, U14 TPS2557DRBR, U16 TPS2557DRBR, U17 TPS2557DRBR, U18 TPS2557DRBR, U19 TPS2557DRBR

Commit message: .
Parts:
- C_IN10, C_IN6, C_IN7, C_IN8, C_IN9: JLC Part Number (none) -> C338036
- J11, J12, J7, J8, J9: JLC Part Number (none) -> C9900031531
- R40, R43, R45, R48, R50: JLC Part Number (none) -> C3930971
- U14, U16, U17, U18, U19: JLC Part Number (none) -> C130056

Commit message: w
Parts:
- U14, U16, U17, U18, U19: footprint TPS2557:DRB8_2P4X1P65 -> DRB8_2P4X1P65
Changed lines of the file:
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@@
 			)
 		)
-		(property "Footprint" "TPS2557:DRB8_2P4X1P65"
+		(property "Footprint" "DRB8_2P4X1P65"
 			(at 199.39 120.65 0)
 			(effects
@@
 			)
 		)
-		(property "Footprint" "TPS2557:DRB8_2P4X1P65"
+		(property "Footprint" "DRB8_2P4X1P65"
 			(at 62.23 90.17 0)
 			(effects
@@
 			)
 		)
-		(property "Footprint" "TPS2557:DRB8_2P4X1P65"
+		(property "Footprint" "DRB8_2P4X1P65"
 			(at 256.54 121.92 0)
 			(effects
@@
 			)
 		)
-		(property "Footprint" "TPS2557:DRB8_2P4X1P65"
+		(property "Footprint" "DRB8_2P4X1P65"
 			(at 58.42 140.97 0)
 			(effects
@@
 			)
 		)
-		(property "Footprint" "TPS2557:DRB8_2P4X1P65"
+		(property "Footprint" "DRB8_2P4X1P65"
 			(at 64.77 39.37 0)
 			(effects

Commit message: Relabeling according to standards
Parts:
- U701: renamed from U14; footprint DRB8_2P4X1P65 -> (none)
- U702: renamed from U16; footprint DRB8_2P4X1P65 -> (none)
- U703: renamed from U17; footprint DRB8_2P4X1P65 -> (none)
- U704: renamed from U19; footprint DRB8_2P4X1P65 -> (none)
- U705: renamed from U18; footprint DRB8_2P4X1P65 -> (none)
- renumbered C_IN6 to C701, C_OUT11 to C702, C_IN7 to C703, C_OUT12 to C704, C_IN8 to C705, C_OUT13 to C706, C_IN10 to C707, C_OUT15 to C708, C_IN9 to C709, C_OUT14 to C710, J13 to J701, J9 to J702, J14 to J703, J7 to J704, J15 to J705, J8 to J706, J17 to J707, J12 to J708, J16 to J709, J11 to J710, R40 to R701, R39 to R702, R43 to R703, R42 to R704, R45 to R705, R44 to R706, R50 to R707, R49 to R708, R48 to R709, R47 to R710
Connections:
- net OCPC_ADCS_ENABLE: now also R705.1
