File: PCB1 PANEL_IN SPV1040 BUCK5 BUCK33 OCPC/OCPC.kicad_sch (KiCad schematic)
At the start: 0 parts

Commit message: 2
Other:
- company: (none) -> TEAM ANANT
Changed lines of the file:
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@@
 	(generator_version "8.0")
 	(paper "A4")
+	(title_block
+		(company "TEAM ANANT")
+		(comment 1 "BITS PILANI")
+	)
 )

Commit message: EDITS
Parts:
- added C_IN6: 0.1uF, Capacitor_SMD:C_0603_1608Metric, symbol Device:C
- added C_OUT11, C_retry1: C, Capacitor_SMD:C_0504_1310Metric, symbol Device:C
- added J7, J9: Conn_01x02_Pin, Connector_PinHeader_2.54mm:PinHeader_1x02_P2.54mm_Vertical, symbol Connector:Conn_01x02_Pin
- added J8: Conn_01x01_Pin, Connector_PinHeader_2.54mm:PinHeader_1x01_P2.54mm_Vertical, symbol Connector:Conn_01x01_Pin
- added R39: 1k, Resistor_SMD:R_1812_4532Metric, symbol Device:R
- added R_FAULT1: 0-500k, symbol Device:R_Potentiometer
- added R_ILIM1: 0-200k, symbol Device:R_Potentiometer
- added U14: TPS2557DRBR, TPS2557:DRB8_2P4X1P65, symbol TPS2557:TPS2557DRBR
Connections:
- new net: C_OUT11.2, J9.2 (Pin_2), U14.7 (OUT)
- new net: R_ILIM1.1, U14.5 (ILIM)
- new net: R39.1, U14.8 (*FAULT)
- new net EN: C_retry1.1, J8.1 (Pin_1), R39.2, R_FAULT1.3, U14.4 (EN)
- new net GND: C_IN6.1, C_OUT11.1, C_retry1.2, J7.2 (Pin_2), J9.1 (Pin_1), R_ILIM1.2, U14.1 (GND), U14.9 (EPAD)
- new net IN: C_IN6.2, J7.1 (Pin_1), R_FAULT1.2, U14.2 (IN)
- no-connect marks 0 -> 4

Commit message: EDITS NTH
Parts:
- removed C_retry1: C, Capacitor_SMD:C_0504_1310Metric, symbol Device:C
- removed J8: Conn_01x01_Pin, Connector_PinHeader_2.54mm:PinHeader_1x01_P2.54mm_Vertical, symbol Connector:Conn_01x01_Pin
- removed R_FAULT1: 0-500k, symbol Device:R_Potentiometer
- removed R_ILIM1: 0-200k, symbol Device:R_Potentiometer
- added C_IN10, C_IN7, C_IN8, C_IN9: 0.1uF, Capacitor_SMD:C_0603_1608Metric, symbol Device:C
- added C_OUT12, C_OUT13, C_OUT14, C_OUT15: 100uF, Capacitor_SMD:C_0504_1310Metric, symbol Device:C
- added J11, J12, J8: Conn_01x02_Pin, Connector_PinHeader_2.54mm:PinHeader_1x02_P2.54mm_Vertical, symbol Connector:Conn_01x02_Pin
- added R40, R43, R45, R48, R50: 100k, Resistor_SMD:R_01005_0402Metric_Pad0.57x0.30mm_HandSolder, symbol Device:R
- added R42, R44, R47, R49: R, Resistor_SMD:R_0603_1608Metric_Pad0.98x0.95mm_HandSolder, symbol Device:R
- added U16, U17, U18, U19: TPS2557DRBR, TPS2557:DRB8_2P4X1P65, symbol TPS2557:TPS2557DRBR
- C_OUT11: value C -> 100uF
- R39: value 1k -> R; footprint Resistor_SMD:R_1812_4532Metric -> Resistor_SMD:R_0603_1608Metric_Pad0.98x0.95mm_HandSolder
Connections:
- net GND: now also J7.1 (Pin_1), R39.2, C_IN10.1, C_IN7.1, C_IN8.1, C_IN9.1, C_OUT12.1, C_OUT13.1, C_OUT14.1, C_OUT15.1, J11.1 (Pin_1), J12.1 (Pin_1), J8.1 (Pin_1), R42.2, R44.2, R47.2, R49.2, U16.1 (GND), U16.9 (EPAD), U17.1 (GND), U17.9 (EPAD), U18.1 (GND), U18.9 (EPAD), U19.1 (GND), U19.9 (EPAD); no longer J7.2 (Pin_2)
- net IN: now also C_IN10.2, C_IN7.2, C_IN8.2, C_IN9.2, R40.1, R43.1, R45.1, R48.1, R50.1, U16.2 (IN), U17.2 (IN), U18.2 (IN), U19.2 (IN); no longer J7.1 (Pin_1)
- net at U14.5 (ILIM): now also R39.1
- net OCPC_1_FAULT: now reaches U14.8 (*FAULT)
- net OCPC_1_FAULT: now also R40.2, R43.2, R45.2, R48.2, R50.2, U16.8 (*FAULT), U17.8 (*FAULT), U18.8 (*FAULT), U19.8 (*FAULT); no longer R39.1
- net EN renamed OCPC_1_EN
- net OCPC_1_EN: now also U16.4 (EN), U17.4 (EN), U18.4 (EN), U19.4 (EN); no longer R39.2
- new net: R47.1, U18.5 (ILIM)
- new net: R44.1, U17.5 (ILIM)
- new net: C_OUT13.2, J8.2 (Pin_2), U17.7 (OUT)
- new net: R49.1, U19.5 (ILIM)
- new net: C_OUT14.2, J11.2 (Pin_2), U18.7 (OUT)
- new net: C_OUT15.2, J12.2 (Pin_2), U19.7 (OUT)
- new net: R42.1, U16.5 (ILIM)
- new net: C_OUT12.2, J7.2 (Pin_2), U16.7 (OUT)
- no-connect marks 4 -> 10
Other:
- note added: "REMOVED AUTO-RETRY FEATURE"
- note added: "REMOVED AUTO-RETRY FEATURE OBC"
- moved on the sheet: C_IN6, C_OUT11, J9, U14

Commit message: EDITS N+1
Parts:
- added J13, J14, J15, J16, J17: OCPC_EN, symbol Connector:Conn_01x01_Pin
Connections:
- net OCPC_1_EN: now also J13.1 (Pin_1), J14.1 (Pin_1), J15.1 (Pin_1), J16.1 (Pin_1), J17.1 (Pin_1)

Commit message: s
Connections:
- net 3.3V_ADCS_OCPC: now reaches C_OUT13.2, J8.2 (Pin_2), U17.7 (OUT)
- net 3.3V_TTC_OCPC: now reaches C_OUT14.2, J11.2 (Pin_2), U18.7 (OUT)
- net 5V_PAYLOAD_OCPC: now reaches C_OUT15.2, J12.2 (Pin_2), U19.7 (OUT)
- net 5V_OBC_OCPC: now reaches C_OUT11.2, J9.2 (Pin_2), U14.7 (OUT)
- net 5V_ADCSC_OCPC: now reaches C_OUT12.2, J7.2 (Pin_2), U16.7 (OUT)
- removed net IN: C_IN10.2, C_IN6.2, C_IN7.2, C_IN8.2, C_IN9.2, R40.1, R43.1, R45.1, R48.1, R50.1, U14.2 (IN), U16.2 (IN), U17.2 (IN), U18.2 (IN), U19.2 (IN)
- removed net OCPC_1_EN: J13.1 (Pin_1), J14.1 (Pin_1), J15.1 (Pin_1), J16.1 (Pin_1), J17.1 (Pin_1), U14.4 (EN), U16.4 (EN), U17.4 (EN), U18.4 (EN), U19.4 (EN)
- removed net OCPC_1_FAULT: R40.2, R43.2, R45.2, R48.2, R50.2, U14.8 (*FAULT), U16.8 (*FAULT), U17.8 (*FAULT), U18.8 (*FAULT), U19.8 (*FAULT)
- new net 3.3V_ADCS: C_IN8.2, U17.2 (IN)
- new net 3.3v_TTC: C_IN9.2, U18.2 (IN)
- new net 5V_ADCSC: C_IN7.2, U16.2 (IN)
- new net 5V_OBC: C_IN6.2, U14.2 (IN)
- new net 5V_PAYLOAD: C_IN10.2, U19.2 (IN)
- new net OCPC_ADCSC_ENABLE: J14.1 (Pin_1), R43.1, U16.4 (EN)
- new net OCPC_ADCSC_FAULT: R43.2, U16.8 (*FAULT)
- new net OCPC_ADCS_ENABLE: J15.1 (Pin_1), U17.4 (EN)
- new net OCPC_ADCS_FAULT: R45.2, U17.8 (*FAULT)
- new net OCPC_OBC_ENABLE: J13.1 (Pin_1), R40.1, U14.4 (EN)
- new net OCPC_OBC_FAULT: R40.2, U14.8 (*FAULT)
- new net OCPC_PAYLOAD_ENABLE: J17.1 (Pin_1), R50.1, U19.4 (EN)
- new net OCPC_PAYLOAD_FAULT: R50.2, U19.8 (*FAULT)
- new net OCPC_TTC_ENABLE: J16.1 (Pin_1), R48.1, U18.4 (EN)
- new net OCPC_TTC_FAULT: R48.2, U18.8 (*FAULT)

Commit message: VCOMMIT
EDITS N+I
Parts:
- removed C_IN6, C_IN7, C_IN8: 0.1uF, Capacitor_SMD:C_0603_1608Metric, symbol Device:C
- removed C_OUT11, C_OUT12, C_OUT13: 100uF, Capacitor_SMD:C_0504_1310Metric, symbol Device:C
- removed J13, J14, J15: OCPC_EN, symbol Connector:Conn_01x01_Pin
- removed J7, J8, J9: Conn_01x02_Pin, Connector_PinHeader_2.54mm:PinHeader_1x02_P2.54mm_Vertical, symbol Connector:Conn_01x02_Pin
- removed R39, R42, R44: R, Resistor_SMD:R_0603_1608Metric_Pad0.98x0.95mm_HandSolder, symbol Device:R
- removed R40, R43, R45: 100k, Resistor_SMD:R_01005_0402Metric_Pad0.57x0.30mm_HandSolder, symbol Device:R
- removed U14, U16, U17: TPS2557DRBR, TPS2557:DRB8_2P4X1P65, symbol TPS2557:TPS2557DRBR
Connections:
- no-connect marks 10 -> 4
Other:
- note removed: "REMOVED AUTO-RETRY FEATURE OBC"
