File: PCB1 PANEL_IN SPV1040 BUCK5 BUCK33 OCPC/USB_CHARGER_DEPRECATED.kicad_sch (KiCad schematic)
At the start: 17 parts, among them J1 Conn_01x06, J10 USB_C_Receptacle_USB2.0_16P, U1 BQ25883RGER

Commit message: Relabeling according to standards
Parts:
- renumbered C1 to C201, C3 to C202, C2 to C203, C4 to C204, C7 to C205, C5 to C206, C6 to C207, D1 to D201, J10 to J201, J1 to J202, L1 to L201, R2 to R201, R3 to R202, R4 to R203, R6 to R204, R5 to R205, U1 to U201
Changed lines of the file:
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@@
 		(on_board yes)
 		(dnp no)
-		(property "Reference" "C1"
+		(property "Reference" "C201"
 			(at 132.08 63.5 0)
 			(effects
@@
 			(project "PCB1 PANEL_IN SPV1040 BUCK5 BUCK33 OCPC"
 				(path "/494c9d9f-6b33-4248-a813-27ffaaa929bd/d0756281-183d-4749-b648-78cca7febb2e"
-					(reference "C1")
+					(reference "C201")
 					(unit 1)
 				)
@@
 		(on_board yes)
 		(dnp no)
-		(property "Reference" "C6"
+		(property "Reference" "C207"
 			(at 185.2168 96.6216 0)
 			(effects
@@
 			(project "PCB1 PANEL_IN SPV1040 BUCK5 BUCK33 OCPC"
 				(path "/494c9d9f-6b33-4248-a813-27ffaaa929bd/d0756281-183d-4749-b648-78cca7febb2e"
-					(reference "C6")
+					(reference "C207")
 					(unit 1)
 				)
@@
 		(on_board yes)
 		(dnp no)
-		(property "Reference" "R2"
+		(property "Reference" "R201"
 			(at 131.6482 111.8616 0)
 			(effects
@@
 			(project "PCB1 PANEL_IN SPV1040 BUCK5 BUCK33 OCPC"
 				(path "/494c9d9f-6b33-4248-a813-27ffaaa929bd/d0756281-183d-4749-b648-78cca7febb2e"
-					(reference "R2")
+					(reference "R201")
 					(unit 1)
 				)
@@
 		(on_board yes)
 		(dnp no)
-		(property "Reference" "C4"
+		(property "Reference" "C204"
 			(at 172.72 111.0234 90)
 			(effects
@@
 			(project "PCB1 PANEL_IN SPV1040 BUCK5 BUCK33 OCPC"
 				(path "/494c9d9f-6b33-4248-a813-27ffaaa929bd/d0756281-183d-4749-b648-78cca7febb2e"
-					(reference "C4")
+					(reference "C204")
 					(unit 1)
 				)
@@
 		(on_board yes)
 		(dnp no)
-		(property "Reference" "C7"
+		(property "Reference" "C205"
 			(at 180.34 107.95 0)
 			(effects
@@
 			(project "PCB1 PANEL_IN SPV1040 BUCK5 BUCK33 OCPC"
 				(path "/494c9d9f-6b33-4248-a813-27ffaaa929bd/d0756281-183d-4749-b648-78cca7febb2e"
-					(reference "C7")
+					(reference "C205")
 					(unit 1)
 				)
@@
 		(dnp no)
 		(fields_autoplaced yes)
-		(property "Reference" "J10"
+		(property "Reference" "J201"
 			(at 86.36 74.93 0)
 			(effects
@@
 			(project "PCB1 PANEL_IN SPV1040 BUCK5 BUCK33 OCPC"
 				(path "/494c9d9f-6b33-4248-a813-27ffaaa929bd/d0756281-183d-4749-b648-78cca7febb2e"
-					(reference "J10")
+					(reference "J201")
 					(unit 1)
 				)
@@
 		(on_board yes)
 		(dnp no)
-		(property "Reference" "D1"
+		(property "Reference" "D201"
 			(at 169.0878 119.3546 0)
 			(effects
@@
 			(project "PCB1 PANEL_IN SPV1040 BUCK5 BUCK33 OCPC"
 				(path "/494c9d9f-6b33-4248-a813-27ffaaa929bd/d0756281-183d-4749-b648-78cca7febb2e"
-					(reference "D1")
+					(reference "D201")
 					(unit 1)
 				)
@@
 		(on_board yes)
 		(dnp no)
-		(property "Reference" "J1"
+		(property "Reference" "J202"
 			(at 204.1652 71.9328 90)
 			(effects
@@
 			(project "PCB1 PANEL_IN SPV1040 BUCK5 BUCK33 OCPC"
 				(path "/494c9d9f-6b33-4248-a813-27ffaaa929bd/d0756281-183d-4749-b648-78cca7febb2e"
-					(reference "J1")
+					(reference "J202")
 					(unit 1)
 				)
@@
 		(on_board yes)
 		(dnp no)
-		(property "Reference" "C2"
+		(property "Reference" "C203"
 			(at 137.16 127 90)
 			(effects
@@
 			(project "PCB1 PANEL_IN SPV1040 BUCK5 BUCK33 OCPC"
 				(path "/494c9d9f-6b33-4248-a813-27ffaaa929bd/d0756281-183d-4749-b648-78cca7febb2e"
-					(reference "C2")
+					(reference "C203")
 					(unit 1)
 				)
@@
 		(on_board yes)
 		(dnp no)
-		(property "Reference" "U1"
+		(property "Reference" "U201"
 			(at 153.67 87.63 0)
 			(effects
@@
 			(project "PCB1 PANEL_IN SPV1040 BUCK5 BUCK33 OCPC"
 				(path "/494c9d9f-6b33-4248-a813-27ffaaa929bd/d0756281-183d-4749-b648-78cca7febb2e"
-					(reference "U1")
+					(reference "U201")
 					(unit 1)
 				)
@@
 		(on_board yes)
 		(dnp no)
-		(property "Reference" "C3"
+		(property "Reference" "C202"
 			(at 163.83 63.5 0)
 			(effects
@@
 			(project "PCB1 PANEL_IN SPV1040 BUCK5 BUCK33 OCPC"
 				(path "/494c9d9f-6b33-4248-a813-27ffaaa929bd/d0756281-183d-4749-b648-78cca7febb2e"
-					(reference "C3")
+					(reference "C202")
 					(unit 1)
 				)
@@
 		(on_board yes)
 		(dnp no)
-		(property "Reference" "R6"
+		(property "Reference" "R204"
 			(at 161.29 119.253 90)
 			(effects
@@
 			(project "PCB1 PANEL_IN SPV1040 BUCK5 BUCK33 OCPC"
 				(path "/494c9d9f-6b33-4248-a813-27ffaaa929bd/d0756281-183d-4749-b648-78cca7febb2e"
-					(reference "R6")
+					(reference "R204")
 					(unit 1)
 				)
@@
 		(on_board yes)
 		(dnp no)
-		(property "Reference" "R4"
+		(property "Reference" "R203"
 			(at 138.8872 119.4816 0)
 			(effects
@@
 			(project "PCB1 PANEL_IN SPV1040 BUCK5 BUCK33 OCPC"
 				(path "/494c9d9f-6b33-4248-a813-27ffaaa929bd/d0756281-183d-4749-b648-78cca7febb2e"
-					(reference "R4")
+					(reference "R203")
 					(unit 1)
 				)
@@
 		(on_board yes)
 		(dnp no)
-		(property "Reference" "L1"
+		(property "Reference" "L201"
 			(at 175.26 87.63 0)
 			(effects
@@
 			(project "PCB1 PANEL_IN SPV1040 BUCK5 BUCK33 OCPC"
 				(path "/494c9d9f-6b33-4248-a813-27ffaaa929bd/d0756281-183d-4749-b648-78cca7febb2e"
-					(reference "L1")
+					(reference "L201")
 					(unit 1)
 				)
@@
 		(on_board yes)
 		(dnp no)
-		(property "Reference" "R5"
+		(property "Reference" "R205"
 			(at 146.05 135.89 90)
 			(effects
@@
 			(project "PCB1 PANEL_IN SPV1040 BUCK5 BUCK33 OCPC"
 				(path "/494c9d9f-6b33-4248-a813-27ffaaa929bd/d0756281-183d-4749-b648-78cca7febb2e"
-					(reference "R5")
+					(reference "R205")
 					(unit 1)
 				)
@@
 		(on_board yes)
 		(dnp no)
-		(property "Reference" "R3"
+		(property "Reference" "R202"
 			(at 131.6482 119.4816 0)
 			(effects
@@
 			(project "PCB1 PANEL_IN SPV1040 BUCK5 BUCK33 OCPC"
 				(path "/494c9d9f-6b33-4248-a813-27ffaaa929bd/d0756281-183d-4749-b648-78cca7febb2e"
-					(reference "R3")
+					(reference "R202")
 					(unit 1)
 				)
@@
 		(on_board yes)
 		(dnp no)
-		(property "Reference" "C5"
+		(property "Reference" "C206"
 			(at 176.53 96.52 0)
 			(effects
@@
 			(project "PCB1 PANEL_IN SPV1040 BUCK5 BUCK33 OCPC"
 				(path "/494c9d9f-6b33-4248-a813-27ffaaa929bd/d0756281-183d-4749-b648-78cca7febb2e"
-					(reference "C5")
-					(unit 1)
-				)
+					(reference "C206")
+					(unit 1)
+				)
