File: PCB1 PANEL_IN SPV1040 BUCK5 BUCK33 OCPC/WATCHDOG.kicad_sch (KiCad schematic)
At the start: 6 parts, among them SW2 KMR231NG LFS, U22 MAX706RESA

Commit message: .
Parts:
- C?: renamed from C52; JLCPCB Part# (none) -> C1592
- R?: renamed from R60; JLCPCB Part# (none) -> C115324
- R?: renamed from R58; JLCPCB Part# (none) -> C115324
- R?: renamed from R59; JLCPCB Part# (none) -> C115324
- SW?: renamed from SW2; JLCPCB Part# (none) -> C221679
- U?: renamed from U22; JLCPCB Part# (none) -> C3687309
Changed lines of the file:
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@@
 		(on_board yes)
 		(dnp no)
-		(property "Reference" "R60"
+		(property "Reference" "R?"
 			(at 212.09 120.015 0)
 			(effects
@@
 			)
 		)
+		(property "JLCPCB Part#" "C115324"
+			(at 209.55 121.285 0)
+			(effects
+				(font
+					(size 1.27 1.27)
+				)
+				(hide yes)
+			)
+		)
 		(pin "1"
 		)
@@
 		)
 		(instances
+			(project "WATCHDOG"
+				(path "/2de3fe5d-6388-4a09-bd44-13c721b25522"
+					(reference "R?")
+					(unit 1)
+				)
+			)
 			(project "PCB1 PANEL_IN SPV1040 BUCK5 BUCK33 OCPC"
 				(path "/494c9d9f-6b33-4248-a813-27ffaaa929bd/8cd5401d-8e6e-4c5c-abb2-269e996089da"
@@
 		(on_board yes)
 		(dnp no)
-		(property "Reference" "R58"
+		(property "Reference" "R?"
 			(at 176.53 93.345 0)
 			(effects
@@
 			)
 		)
+		(property "JLCPCB Part#" "C115324"
+			(at 180.34 94.615 0)
+			(effects
+				(font
+					(size 1.27 1.27)
+				)
+				(hide yes)
+			)
+		)
 		(pin "1"
 		)
@@
 		)
 		(instances
+			(project "WATCHDOG"
+				(path "/2de3fe5d-6388-4a09-bd44-13c721b25522"
+					(reference "R?")
+					(unit 1)
+				)
+			)
 			(project "PCB1 PANEL_IN SPV1040 BUCK5 BUCK33 OCPC"
 				(path "/494c9d9f-6b33-4248-a813-27ffaaa929bd/8cd5401d-8e6e-4c5c-abb2-269e996089da"
@@
 		(on_board yes)
 		(dnp no)
-		(property "Reference" "#GND07"
+		(property "Reference" "#GND?"
 			(at 167.64 135.255 0)
 			(effects
@@
 		)
 		(instances
+			(project "WATCHDOG"
+				(path "/2de3fe5d-6388-4a09-bd44-13c721b25522"
+					(reference "#GND?")
+					(unit 1)
+				)
+			)
 			(project "PCB1 PANEL_IN SPV1040 BUCK5 BUCK33 OCPC"
 				(path "/494c9d9f-6b33-4248-a813-27ffaaa929bd/8cd5401d-8e6e-4c5c-abb2-269e996089da"
@@
 		(on_board yes)
 		(dnp no)
-		(property "Reference" "#SUPPLY04"
+		(property "Reference" "#SUPPLY?"
 			(at 243.84 70.485 0)
 			(effects
@@
 		)
 		(instances
+			(project "WATCHDOG"
+				(path "/2de3fe5d-6388-4a09-bd44-13c721b25522"
+					(reference "#SUPPLY?")
+					(unit 1)
+				)
+			)
 			(project "PCB1 PANEL_IN SPV1040 BUCK5 BUCK33 OCPC"
 				(path "/494c9d9f-6b33-4248-a813-27ffaaa929bd/8cd5401d-8e6e-4c5c-abb2-269e996089da"
@@
 		(on_board yes)
 		(dnp no)
-		(property "Reference" "#GND09"
+		(property "Reference" "#GND?"
 			(at 194.31 132.715 0)
 			(effects
@@
 		)
 		(instances
+			(project "WATCHDOG"
+				(path "/2de3fe5d-6388-4a09-bd44-13c721b25522"
+					(reference "#GND?")
+					(unit 1)
+				)
+			)
 			(project "PCB1 PANEL_IN SPV1040 BUCK5 BUCK33 OCPC"
 				(path "/494c9d9f-6b33-4248-a813-27ffaaa929bd/8cd5401d-8e6e-4c5c-abb2-269e996089da"
@@
 		(on_board yes)
 		(dnp no)
-		(property "Reference" "U22"
+		(property "Reference" "U?"
 			(at 210.82 70.2818 0)
 			(effects
@@
 			)
 		)
-		(property "JLCPCB Part#" ""
+		(property "JLCPCB Part#" "C3687309"
 			(at 231.14 80.645 0)
 			(effects
@@
 		)
 		(instances
+			(project "WATCHDOG"
+				(path "/2de3fe5d-6388-4a09-bd44-13c721b25522"
+					(reference "U?")
+					(unit 1)
+				)
+			)
 			(project "PCB1 PANEL_IN SPV1040 BUCK5 BUCK33 OCPC"
 				(path "/494c9d9f-6b33-4248-a813-27ffaaa929bd/8cd5401d-8e6e-4c5c-abb2-269e996089da"
@@
 		(on_board yes)
 		(dnp no)
-		(property "Reference" "R59"
+		(property "Reference" "R?"
 			(at 200.66 120.015 0)
 			(effects
@@
 			)
 		)
+		(property "JLCPCB Part#" "C115324"
+			(at 204.47 121.285 0)
+			(effects
+				(font
+					(size 1.27 1.27)
+				)
+				(hide yes)
+			)
+		)
 		(pin "1"
 		)
@@
 		)
 		(instances
+			(project "WATCHDOG"
+				(path "/2de3fe5d-6388-4a09-bd44-13c721b25522"
+					(reference "R?")
+					(unit 1)
+				)
+			)
 			(project "PCB1 PANEL_IN SPV1040 BUCK5 BUCK33 OCPC"
 				(path "/494c9d9f-6b33-4248-a813-27ffaaa929bd/8cd5401d-8e6e-4c5c-abb2-269e996089da"
@@
 		(on_board yes)
 		(dnp no)
-		(property "Reference" "#GND08"
+		(property "Reference" "#GND?"
 			(at 193.04 100.965 0)
 			(effects
@@
 		)
 		(instances
+			(project "WATCHDOG"
+				(path "/2de3fe5d-6388-4a09-bd44-13c721b25522"
+					(reference "#GND?")
+					(unit 1)
+				)
+			)
 			(project "PCB1 PANEL_IN SPV1040 BUCK5 BUCK33 OCPC"
 				(path "/494c9d9f-6b33-4248-a813-27ffaaa929bd/8cd5401d-8e6e-4c5c-abb2-269e996089da"
@@
 		(on_board yes)
 		(dnp no)
-		(property "Reference" "C52"
+		(property "Reference" "C?"
 			(at 191.9732 126.4666 0)
 			(effects
@@
 			)
 		)
+		(property "JLCPCB Part#" "C1592"
+			(at 194.31 127.635 0)
+			(effects
+				(font
+					(size 1.27 1.27)
+				)
+				(hide yes)
+			)
+		)
 		(pin "1"
 		)
@@
 		)
 		(instances
+			(project "WATCHDOG"
+				(path "/2de3fe5d-6388-4a09-bd44-13c721b25522"
+					(reference "C?")
+					(unit 1)
+				)
+			)
 			(project "PCB1 PANEL_IN SPV1040 BUCK5 BUCK33 OCPC"
 				(path "/494c9d9f-6b33-4248-a813-27ffaaa929bd/8cd5401d-8e6e-4c5c-abb2-269e996089da"
@@
 		(on_board yes)
 		(dnp no)
-		(property "Reference" "#GND010"
+		(property "Reference" "#GND?"
 			(at 243.84 100.965 0)
 			(effects
@@
 		)
 		(instances
+			(project "WATCHDOG"
+				(path "/2de3fe5d-6388-4a09-bd44-13c721b25522"
+					(reference "#GND?")
+					(unit 1)
+				)
+			)
 			(project "PCB1 PANEL_IN SPV1040 BUCK5 BUCK33 OCPC"
 				(path "/494c9d9f-6b33-4248-a813-27ffaaa929bd/8cd5401d-8e6e-4c5c-abb2-269e996089da"
@@
 		(on_board yes)
 		(dnp no)
-		(property "Reference" "#SUPPLY03"
+		(property "Reference" "#SUPPLY?"
 			(at 207.01 113.665 0)
 			(effects
@@
 		)
 		(instances
+			(project "WATCHDOG"
+				(path "/2de3fe5d-6388-4a09-bd44-13c721b25522"
+					(reference "#SUPPLY?")
+					(unit 1)
+				)
+			)
 			(project "PCB1 PANEL_IN SPV1040 BUCK5 BUCK33 OCPC"
 				(path "/494c9d9f-6b33-4248-a813-27ffaaa929bd/8cd5401d-8e6e-4c5c-abb2-269e996089da"
@@
 		(on_board yes)
 		(dnp no)
-		(property "Reference" "SW2"
+		(property "Reference" "SW?"
 			(at 173.99 128.905 0)
 			(effects
@@
 			)
 		)
+		(property "JLCPCB Part#" "C221679"
+			(at 172.72 125.095 0)
+			(effects
+				(font
+					(size 1.27 1.27)
+				)
+				(hide yes)
+			)
+		)
 		(pin "A"
 		)
@@
 		)
 		(instances
+			(project "WATCHDOG"
+				(path "/2de3fe5d-6388-4a09-bd44-13c721b25522"
+					(reference "SW?")
+					(unit 1)
+				)
+			)
 			(project "PCB1 PANEL_IN SPV1040 BUCK5 BUCK33 OCPC"
 				(path "/494c9d9f-6b33-4248-a813-27ffaaa929bd/8cd5401d-8e6e-4c5c-abb2-269e996089da"
@@
 		)
 	)
+	(sheet_instances
+		(path "/"
+			(page "1")
+		)
+	)
