File: PCB1 PANEL_IN SPV1040 BUCK5 BUCK33 OCPC/BUCK5.kicad_sch (KiCad schematic)
At the start: 19 parts, among them U7 LM21305SQ/NOPB

Commit message: VCOMMIT
EDITS N+I
Parts:
- removed C27: 2u2, Capacitor_Tantalum_SMD:CP_EIA-7343-43_Kemet-X_Pad2.25x2.55mm_HandSolder, symbol Device:C_Small
- removed C28, C29, C30, C31, C32, C33, C34, C35: 2u2, Capacitor_SMD:C_0603_1608Metric_Pad1.08x0.95mm_HandSolder, symbol Device:C_Small
- removed L7: L, Inductor_SMD:L_6.3x6.3_H3, symbol Device:L
- removed R21, R22, R31, R32, R33, R34, R35, R36: 1k, Resistor_SMD:R_0603_1608Metric_Pad0.98x0.95mm_HandSolder, symbol Device:R_Small
- removed U7: LM21305SQ/NOPB, footprintLM21305:LM21305SQ&slash_NOPB, symbol 2023-03-29_16-01-02:LM21305SQ/NOPB
Other:
- note removed: "MAKE THIS INTO 5V"
