File: PCB1 PANEL_IN SPV1040 BUCK5 BUCK33 OCPC/MSP430.kicad_sch (KiCad schematic)
At the start: 15 parts, among them U20 MSP430F5529IPN, Y1 32K, Y2 CSTCR4M00G53-R0

Commit message: VCOMMIT
EDITS N+I
Parts:
- removed C41, C43, C44, C48: 1u0, Capacitor_SMD:C_0603_1608Metric, symbol Device:C_Small
- removed C42: 10u, Capacitor_SMD:CP_Elec_3x5.3, symbol Device:C_Polarized_Small
- removed C45, C46: 1u1, Capacitor_SMD:C_0603_1608Metric, symbol Device:C_Small
- removed C47, C49: 1u0, Capacitor_SMD:C_0402_1005Metric_Pad0.74x0.62mm_HandSolder, symbol Device:C_Small
- removed C50: 10u, Capacitor_SMD:CP_Elec_4x3.9, symbol Device:C_Polarized_Small
- removed R52: 10k, Resistor_SMD:R_0603_1608Metric, symbol mainboard:R-US_R0603
- removed R53: 10K, Resistor_SMD:R_0603_1608Metric, symbol Device:R_Small
- removed U20: MSP430F5529IPN, footprintMSP:MSP430F5529IPN, symbol 2023-03-28_15-31-46:MSP430F5529IPN
- removed Y1: 32K, Crystal:Crystal_AT310_D3.0mm_L10.0mm_Horizontal_1EP_style1, symbol Device:Crystal_GND2_Small
- removed Y2: CSTCR4M00G53-R0, CSTCR4M00G53-R0:OSC_CSTCR4M00G53-R0, symbol CSTCR4M00G53-R0:CSTCR4M00G53-R0
- added J2-J1, J3-J1: Conn_01x10, Connector_PinSocket_2.54mm:PinSocket_2x10_P2.54mm_Vertical, symbol Connector_Generic:Conn_02x10_Odd_Even
- added R26, R27: 10k, Resistor_SMD:R_0603_1608Metric, symbol Device:R
Connections:
- net GND: now also J2-J1.2 (Pin_2), J3-J1.4 (Pin_4)
- new net *D19: J2-J1.4 (Pin_4)
- new net *D37: J2-J1.7 (Pin_7)
- new net *D38: J2-J1.5 (Pin_5)
- new net *D39: J2-J1.3 (Pin_3)
- new net *D40: J2-J1.1 (Pin_1)
- new net +3V3: J3-J1.1 (Pin_1)
- new net +5V: J3-J1.2 (Pin_2)
- new net D10/SDA: J3-J1.19 (Pin_19)
- new net D11: J2-J1.20 (Pin_20)
- new net D12/SPI.CS: J2-J1.18 (Pin_18)
- new net D13/SPI.CS: J2-J1.16 (Pin_16)
- new net D14/SPI.MISO: J2-J1.14 (Pin_14)
- new net D15/SPI.MOSI: J2-J1.12 (Pin_12)
- new net D17: J2-J1.8 (Pin_8)
- new net D18/SPI.CS: J2-J1.6 (Pin_6)
- new net D23/ADC: J3-J1.6 (Pin_6)
- new net D24/ADC: J3-J1.8 (Pin_8)
- new net D25/ADC: J3-J1.10 (Pin_10)
- new net D26/ADC: J3-J1.12 (Pin_12)
- new net D27/ADC: J3-J1.14 (Pin_14)
- new net D28/ADC: J3-J1.16 (Pin_16)
- new net D29/DAC: J3-J1.18 (Pin_18)
- new net D2/ADC: J3-J1.3 (Pin_3)
- new net D30/DAC: J3-J1.20 (Pin_20)
- new net D31: J2-J1.19 (Pin_19)
- new net D32: J2-J1.17 (Pin_17)
- new net D33: J2-J1.15 (Pin_15)
- new net D34: J2-J1.13 (Pin_13)
- new net D35/TC: J2-J1.11 (Pin_11)
- new net D36/TC: J2-J1.9 (Pin_9)
- new net D3/UART.RX: J3-J1.5 (Pin_5)
- new net D4/UART.TX: J3-J1.7 (Pin_7)
- new net D5: J3-J1.9 (Pin_9)
- new net D6/ADC: J3-J1.11 (Pin_11)
- new net D7/SPI.CLK: J3-J1.13 (Pin_13)
- new net D8: J3-J1.15 (Pin_15)
- new net D9/SCL: J3-J1.17 (Pin_17)
- new net RST/D16: J2-J1.10 (Pin_10)
- new net SCL_0: R27.1
- new net SDA_0: R26.2
- new net VCC: R26.1, R27.2
