File: PCB1 PANEL_IN SPV1040 BUCK5 BUCK33 OCPC/PCB1 PANEL_IN SPV1040 BUCK5 BUCK33 OCPC.kicad_sch (KiCad schematic)
At the start: 0 parts

Commit message: EDITS
Other:
- added sheet INA219 (INA219.kicad_sch)
- added sheet LTC2896 (LTC2896.kicad_sch)
Changed lines of the file:
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@@
+	)
+	(sheet
+		(at 170.18 85.09)
+		(size 12.7 3.81)
+		(fields_autoplaced yes)
+		(stroke
+			(width 0.1524)
+			(type solid)
+		)
+		(fill
+			(color 0 0 0 0.0000)
+		)
+		(property "Sheetname" "LTC2896"
+			(at 170.18 84.3784 0)
+			(effects
+				(font
+					(size 1.27 1.27)
+				)
+				(justify left bottom)
+			)
+		)
+		(property "Sheetfile" "LTC2896.kicad_sch"
+			(at 170.18 89.4846 0)
+			(effects
+				(font
+					(size 1.27 1.27)
+				)
+				(justify left top)
+			)
+		)
+		(instances
+			(project "PCB1 PANEL_IN SPV1040 BUCK5 BUCK33 OCPC"
+				(path "/494c9d9f-6b33-4248-a813-27ffaaa929bd"
+					(page "12")
+				)
+			)
+		)
 	)
 	(sheet
@@
 				)
 			)
+		)
+	)
+	(sheet
+		(at 158.75 135.89)
+		(size 12.7 3.81)
+		(fields_autoplaced yes)
+		(stroke
+			(width 0.1524)
+			(type solid)
+		)
+		(fill
+			(color 0 0 0 0.0000)
+		)
+		(property "Sheetname" "INA219"
+			(at 158.75 135.1784 0)
+			(effects
+				(font
+					(size 1.27 1.27)
+				)
+				(justify left bottom)
+			)
+		)
+		(property "Sheetfile" "INA219.kicad_sch"
+			(at 158.75 140.2846 0)
+			(effects
+				(font
+					(size 1.27 1.27)
+				)
+				(justify left top)
+			)
+		)
+		(instances
+			(project "PCB1 PANEL_IN SPV1040 BUCK5 BUCK33 OCPC"
+				(path "/494c9d9f-6b33-4248-a813-27ffaaa929bd"
+					(page "13")
+				)
+			)

Commit message: EDITS NTH
Other:
- sheet LTC2896 renamed LTC2986
- sheet USB_CHARGER renamed USB_CHARGER DEPRECATED
- added sheet RS422 (RS422.kicad_sch)
- sheet LTC2986: file LTC2896.kicad_sch -> LTC2986.kicad_sch
- sheet USB_CHARGER DEPRECATED: file USB_CHARGER.kicad_sch -> USB_CHARGER_DEPRECATED.kicad_sch
Changed lines of the file:
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@@
 	(paper "A4")
 	(title_block
+		(date "V1")
 		(company "TEAM ANANT")
 		(comment 1 "BITS PILANI")
@@
 			(color 0 0 0 0.0000)
 		)
-		(property "Sheetname" "LTC2896"
+		(property "Sheetname" "LTC2986"
 			(at 170.18 84.3784 0)
 			(effects
@@
 			)
 		)
-		(property "Sheetfile" "LTC2896.kicad_sch"
+		(property "Sheetfile" "LTC2986.kicad_sch"
 			(at 170.18 89.4846 0)
 			(effects
@@
 				)
 				(justify left top)
+				(hide yes)
 			)
 		)
@@
 			(color 0 0 0 0.0000)
 		)
-		(property "Sheetname" "USB_CHARGER"
+		(property "Sheetname" "USB_CHARGER DEPRECATED"
 			(at 133.35 37.3884 0)
 			(effects
@@
 			)
 		)
-		(property "Sheetfile" "USB_CHARGER.kicad_sch"
+		(property "Sheetfile" "USB_CHARGER_DEPRECATED.kicad_sch"
 			(at 133.35 42.4946 0)
 			(effects
@@
 				)
 			)
+		)
+	)
+	(sheet
+		(at 204.47 129.54)
+		(size 12.7 3.81)
+		(fields_autoplaced yes)
+		(stroke
+			(width 0.1524)
+			(type solid)
+		)
+		(fill
+			(color 0 0 0 0.0000)
+		)
+		(property "Sheetname" "RS422"
+			(at 204.47 128.8284 0)
+			(effects
+				(font
+					(size 1.27 1.27)
+				)
+				(justify left bottom)
+			)
+		)
+		(property "Sheetfile" "RS422.kicad_sch"
+			(at 204.47 133.9346 0)
+			(effects
+				(font
+					(size 1.27 1.27)
+				)
+				(justify left top)
+			)
+		)
+		(property "Field2" ""
+			(at 204.47 129.54 0)
+			(effects
+				(font
+					(size 1.27 1.27)
+				)
+				(hide yes)
+			)
+		)
+		(instances
+			(project "PCB1 PANEL_IN SPV1040 BUCK5 BUCK33 OCPC"
+				(path "/494c9d9f-6b33-4248-a813-27ffaaa929bd"
+					(page "14")
+				)
+			)

Commit message: EDITS N+1
Other:
- added sheet BEACON (BEACON.kicad_sch)
- added sheet BUS_AND_PROTEC (DATA_BUS.kicad_sch)
- added sheet LEVEL_SHIFTER (LEVEL_SHIFTER.kicad_sch)
- added sheet MSP430 (MSP430.kicad_sch)
- added sheet WATCHDOG (WATCHDOG.kicad_sch)
Changed lines of the file:
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@@
+	)
+	(sheet
+		(at 163.83 111.76)
+		(size 26.035 18.415)
+		(fields_autoplaced yes)
+		(stroke
+			(width 0.1524)
+			(type solid)
+		)
+		(fill
+			(color 0 0 0 0.0000)
+		)
+		(property "Sheetname" "BEACON"
+			(at 163.83 111.0484 0)
+			(effects
+				(font
+					(size 1.27 1.27)
+				)
+				(justify left bottom)
+			)
+		)
+		(property "Sheetfile" "BEACON.kicad_sch"
+			(at 163.83 130.7596 0)
+			(effects
+				(font
+					(size 1.27 1.27)
+				)
+				(justify left top)
+			)
+		)
+		(instances
+			(project "PCB1 PANEL_IN SPV1040 BUCK5 BUCK33 OCPC"
+				(path "/494c9d9f-6b33-4248-a813-27ffaaa929bd"
+					(page "15")
+				)
+			)
+		)
+	)
+	(sheet
+		(at 152.4 156.21)
+		(size 12.7 3.81)
+		(fields_autoplaced yes)
+		(stroke
+			(width 0.1524)
+			(type solid)
+		)
+		(fill
+			(color 0 0 0 0.0000)
+		)
+		(property "Sheetname" "LEVEL_SHIFTER"
+			(at 152.4 155.4984 0)
+			(effects
+				(font
+					(size 1.27 1.27)
+				)
+				(justify left bottom)
+			)
+		)
+		(property "Sheetfile" "LEVEL_SHIFTER.kicad_sch"
+			(at 152.4 160.6046 0)
+			(effects
+				(font
+					(size 1.27 1.27)
+				)
+				(justify left top)
+			)
+		)
+		(instances
+			(project "PCB1 PANEL_IN SPV1040 BUCK5 BUCK33 OCPC"
+				(path "/494c9d9f-6b33-4248-a813-27ffaaa929bd"
+					(page "17")
+				)
+			)
+		)
 	)
 	(sheet
@@
 	)
 	(sheet
+		(at 231.14 54.61)
+		(size 29.21 13.97)
+		(fields_autoplaced yes)
+		(stroke
+			(width 0.1524)
+			(type solid)
+		)
+		(fill
+			(color 0 0 0 0.0000)
+		)
+		(property "Sheetname" "WATCHDOG"
+			(at 231.14 53.8984 0)
+			(effects
+				(font
+					(size 1.27 1.27)
+				)
+				(justify left bottom)
+			)
+		)
+		(property "Sheetfile" "WATCHDOG.kicad_sch"
+			(at 231.14 69.1646 0)
+			(effects
+				(font
+					(size 1.27 1.27)
+				)
+				(justify left top)
+			)
+		)
+		(instances
+			(project "PCB1 PANEL_IN SPV1040 BUCK5 BUCK33 OCPC"
+				(path "/494c9d9f-6b33-4248-a813-27ffaaa929bd"
+					(page "19")
+				)
+			)
+		)
+	)
+	(sheet
+		(at 162.56 54.61)
+		(size 14.605 9.525)
+		(fields_autoplaced yes)
+		(stroke
+			(width 0.1524)
+			(type solid)
+		)
+		(fill
+			(color 0 0 0 0.0000)
+		)
+		(property "Sheetname" "MSP430"
+			(at 162.56 53.8984 0)
+			(show_name yes)
+			(effects
+				(font
+					(size 1.27 1.27)
+				)
+				(justify left bottom)
+			)
+		)
+		(property "Sheetfile" "MSP430.kicad_sch"
+			(at 162.56 64.7196 0)
+			(effects
+				(font
+					(size 1.27 1.27)
+				)
+				(justify left top)
+			)
+		)
+		(instances
+			(project "PCB1 PANEL_IN SPV1040 BUCK5 BUCK33 OCPC"
+				(path "/494c9d9f-6b33-4248-a813-27ffaaa929bd"
+					(page "18")
+				)
+			)
+		)
+	)
+	(sheet
 		(at 132.08 66.04)
 		(size 12.7 3.81)
@@
 				)
 			)
+		)
+	)
+	(sheet
+		(at 232.41 111.76)
+		(size 31.115 11.43)
+		(fields_autoplaced yes)
+		(stroke
+			(width 0.1524)
+			(type solid)
+		)
+		(fill
+			(color 0 0 0 0.0000)
+		)
+		(property "Sheetname" "BUS_AND_PROTEC"
+			(at 232.41 111.0484 0)
+			(effects
+				(font
+					(size 1.27 1.27)
+				)
+				(justify left bottom)
+			)
+		)
+		(property "Sheetfile" "DATA_BUS.kicad_sch"
+			(at 232.41 123.7746 0)
+			(effects
+				(font
+					(size 1.27 1.27)
+				)
+				(justify left top)
+			)
+		)
+		(property "Field2" ""
+			(at 232.41 111.76 0)
+			(effects
+				(font
+					(size 1.27 1.27)
+				)
+				(hide yes)
+			)
+		)
+		(instances
+			(project "PCB1 PANEL_IN SPV1040 BUCK5 BUCK33 OCPC"
+				(path "/494c9d9f-6b33-4248-a813-27ffaaa929bd"
+					(page "16")
+				)
+			)

Commit message: VCOMMIT
EDITS N+I
Other:
- removed sheet INA219
- removed sheet LEVEL_SHIFTER
- removed sheet OCPC
- removed sheet PANEL_IN
- removed sheet SPV1040_1
- removed sheet SPV1040_2
- removed sheet SPV1040_3
- removed sheet SPV1040_4
- removed sheet SPV1040_5
- removed sheet USB_CHARGER DEPRECATED
- added sheet POWER OUT BUSES (POWER_OUT_BUSES.kicad_sch)
- added sheet POWER_IN_BUSES (POWER_IN_BUSES.kicad_sch)
