File: PCB 2 MSP430 BUSMONITOR BEACON WATCHDOG DBUS PROTEC/DATA_BUS.kicad_sch (KiCad schematic)
At the start: 45 parts, among them Q1 BSS138DWQ-7, Q2 MBT2222ADW1T1, Q3 MMDT2907, Q4 BSS138DWQ-7, Q5 MBT2222ADW1T1, Q6 BSS138DWQ-7, Q7 MBT2222ADW1T1, Q8 BSS138DWQ-7, Q9 MBT2222ADW1T1, U1 Payload

Commit message: EDITS NTH
Parts:
- removed R10, R11, R14, R15, R16, R8, R9: 0, Resistor_SMD:R_0603_1608Metric, symbol Device:R_US
- added JP1, JP2, JP3, JP4, JP5, JP6, JP7: SolderJumper_2_Open, Jumper:SolderJumper-2_P1.3mm_Open_RoundedPad1.0x1.5mm, symbol Jumper:SolderJumper_2_Open
Connections:
- net I2C33V_SCL: now also JP3.1 (A)
- net I2C33V_SCL_PROTEC: now also JP3.2 (B)
- net I2C33V_SDA: now also JP4.1 (A)
- net I2C33V_SDA_PROTEC: now also JP4.2 (B)
- net I2C5V_SCL: now also JP1.1 (A)
- net I2C5V_SCL_PROTEC: now also JP1.2 (B)
- net I2C5V_SDA: now also JP2.1 (A)
- net I2C5V_SDA_PROTEC: now also JP2.2 (B)
- net MISO: now also JP5.1 (A), JP6.1 (A), JP7.1 (A)
- net MISO_RF1: now also JP6.2 (B)
- net MISO_RF2: now also JP5.2 (B)
- net MISO_SD: now also JP7.2 (B)

Commit message: EDITS N+1
Parts:
- U1: JLCPCB Part# (none) -> ESQ-126-24-G-D
Changed lines of the file:
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@@
+			)
+		)
+		(property "JLCPCB Part#" "ESQ-126-24-G-D"
+			(at 205.105 60.96 0)
+			(effects
+				(font
+					(size 1.27 1.27)
+				)
+				(hide yes)
 			)
 		)

Commit message: Redisgnated components in PCB2 to make more sense
Parts:
- Q402: renamed from Q1; footprint mainboard:BSS138DWQ-7 -> Package_TO_SOT_SMD:SOT-363_SC-70-6_Handsoldering
- Q404: renamed from Q4; footprint mainboard:BSS138DWQ-7 -> Package_TO_SOT_SMD:SOT-363_SC-70-6_Handsoldering
- Q405: renamed from Q6; footprint mainboard:BSS138DWQ-7 -> Package_TO_SOT_SMD:SOT-363_SC-70-6_Handsoldering
- Q406: renamed from Q8; footprint mainboard:BSS138DWQ-7 -> Package_TO_SOT_SMD:SOT-363_SC-70-6_Handsoldering
- U401: renamed from U1; footprint (none) -> Payload:PC104-Standard
- renumbered C1 to C401, C2 to C402, C3 to C403, C4 to C404, JP1 to JP401, JP2 to JP402, JP3 to JP403, JP4 to JP404, JP5 to JP405, JP6 to JP406, JP7 to JP407, Q2 to Q401, Q5 to Q403, Q7 to Q405, Q9 to Q406, Q3 to Q407, R5 to R401, R6 to R402, R3 to R403, R1 to R404, R7 to R405, R19 to R406, R20 to R407, R18 to R408, R17 to R409, R24 to R41, R21 to R410, R25 to R412, R23 to R413, R22 to R414, R26 to R415, R29 to R416, R30 to R417, R28 to R418, R27 to R419, R31 to R420, R4 to R421, R2 to R422, R12 to R423, R13 to R424

Commit message: Signed-off-by: ARYANTECH123 <ateamxxx101@gmail.com>
Parts:
- renumbered Q405 to Q406, Q406 to Q407, Q406 to Q408, Q407 to Q409
Changed lines of the file:
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@@
 		(on_board yes)
 		(dnp no)
-		(property "Reference" "Q406"
+		(property "Reference" "Q407"
 			(at 97.155 110.109 90)
 			(effects
@@
 			(project "PCB 2 MSP430 BUSMONITOR BEACON WATCHDOG DBUS PROTEC"
 				(path "/04a95c0c-1f2d-49e4-8823-3428ac263eb8/d27be3f9-6033-4951-9896-36f1138da046"
-					(reference "Q406")
+					(reference "Q407")
 					(unit 2)
 				)
@@
 		(on_board yes)
 		(dnp no)
-		(property "Reference" "Q405"
+		(property "Reference" "Q406"
 			(at 37.973 136.6266 0)
 			(effects
@@
 			(project "PCB 2 MSP430 BUSMONITOR BEACON WATCHDOG DBUS PROTEC"
 				(path "/04a95c0c-1f2d-49e4-8823-3428ac263eb8/d27be3f9-6033-4951-9896-36f1138da046"
-					(reference "Q405")
+					(reference "Q406")
 					(unit 2)
 				)
@@
 		(on_board yes)
 		(dnp no)
-		(property "Reference" "Q407"
+		(property "Reference" "Q409"
 			(at 188.595 143.129 90)
 			(effects
@@
 			(project "PCB 2 MSP430 BUSMONITOR BEACON WATCHDOG DBUS PROTEC"
 				(path "/04a95c0c-1f2d-49e4-8823-3428ac263eb8/d27be3f9-6033-4951-9896-36f1138da046"
-					(reference "Q407")
+					(reference "Q409")
 					(unit 1)
 				)
@@
 		(on_board yes)
 		(dnp no)
-		(property "Reference" "Q406"
+		(property "Reference" "Q407"
 			(at 97.155 127.9144 90)
 			(effects
@@
 			(project "PCB 2 MSP430 BUSMONITOR BEACON WATCHDOG DBUS PROTEC"
 				(path "/04a95c0c-1f2d-49e4-8823-3428ac263eb8/d27be3f9-6033-4951-9896-36f1138da046"
-					(reference "Q406")
+					(reference "Q407")
 					(unit 1)
 				)
@@
 		(on_board yes)
 		(dnp no)
-		(property "Reference" "Q405"
+		(property "Reference" "Q406"
 			(at 22.733 131.5466 0)
 			(effects
@@
 			(project "PCB 2 MSP430 BUSMONITOR BEACON WATCHDOG DBUS PROTEC"
 				(path "/04a95c0c-1f2d-49e4-8823-3428ac263eb8/d27be3f9-6033-4951-9896-36f1138da046"
-					(reference "Q405")
+					(reference "Q406")
 					(unit 1)
 				)
@@
 		(on_board yes)
 		(dnp no)
-		(property "Reference" "Q406"
+		(property "Reference" "Q408"
 			(at 76.708 130.9116 0)
 			(effects
@@
 			(project "PCB 2 MSP430 BUSMONITOR BEACON WATCHDOG DBUS PROTEC"
 				(path "/04a95c0c-1f2d-49e4-8823-3428ac263eb8/d27be3f9-6033-4951-9896-36f1138da046"
-					(reference "Q406")
+					(reference "Q408")
 					(unit 1)
 				)
@@
 		(on_board yes)
 		(dnp no)
-		(property "Reference" "Q406"
+		(property "Reference" "Q408"
 			(at 91.948 135.9916 0)
 			(effects
@@
 			(project "PCB 2 MSP430 BUSMONITOR BEACON WATCHDOG DBUS PROTEC"
 				(path "/04a95c0c-1f2d-49e4-8823-3428ac263eb8/d27be3f9-6033-4951-9896-36f1138da046"
-					(reference "Q406")
+					(reference "Q408")
 					(unit 2)
 				)
