File: PCB 2 MSP430 BUSMONITOR BEACON WATCHDOG DBUS PROTEC/PCB 2 MSP430 BUSMONITOR BEACON WATCHDOG DBUS PROTEC.kicad_pcb (KiCad board)
At the start: 2 copper layers, 96 x 89.9 mm, 68 parts, among them Q401 MBT2222ADW1T1, Q402 BSS138DWQ-7, Q403 MBT2222ADW1T1, Q404 BSS138DWQ-7, Q405 MBT2222ADW1T1, Q406 BSS138DWQ-7, Q407 MBT2222ADW1T1, Q408 BSS138DWQ-7, Q409 MMDT2907, U201 MAX706RESA, U202 MAX706RESA, U401 Payload, Y1 32K

Commit message: Signed-off-by: ARYANTECH123 <ateamxxx101@gmail.com>
Parts:
- removed R205: 10K, Resistor_SMD:R_0603_1608Metric
- C202, C403, C404, JP403, JP404, Q405, Q406, Q407, Q408, R204, R206, R41, R412, R413, R414, R415, R416, R417, R418, R419, R420, U202: moved to B.Cu
- moved R203 109.3 mm to (66.5, 30.5)
- moved R202 108.8 mm to (66.5, 28.4)
- moved JP402 105.0 mm to (63.1, 90.0), turned to 90 degrees
- moved C201 103.8 mm to (72.1, 29.5), turned to 90 degrees
- moved R419 103.7 mm to (80.4, 86.5), turned to 180 degrees
- moved JP403 103.3 mm to (64.8, 93.0), turned to -90 degrees
- moved U201 101.4 mm to (66.5, 35.1)
- moved R201 100.3 mm to (72.1, 33.5), turned to -90 degrees
- moved R420 99.6 mm to (73.8, 89.5)
- moved JP404 97.5 mm to (64.5, 86.3), turned to -90 degrees
- moved U202 96.9 mm to (65.0, 48.3), turned to 90 degrees
- moved R418 95.9 mm to (68.1, 85.4), turned to 180 degrees
- moved C202 94.6 mm to (64.0, 42.7)
- moved C7 93.5 mm to (115.0, 29.0)
- moved C10 93.5 mm to (115.0, 34.1)
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Connections:
- C202 pad 2: EPS_RESET -> OBC_RESET
- R204 pad 1: EPS_RESET -> OBC_RESET
- U401 pad 96: EPS_RESET -> OBC_RESET
Routing:
- net I2C33V_SDA_PROTEC: track 0.00 -> 21.7 mm
- net I2C33V_SCL_PROTEC: track 0.00 -> 21.7 mm
- net I2C5V_SDA_PROTEC: track 0.00 -> 17.2 mm
- net OBC_RESET: track 0.00 -> 16.5 mm
- net 3.3V: track 0.00 -> 15.1 mm
- net OBC_WDT_WDI: track 0.00 -> 14.0 mm
- net Net-(Q405B-B2): track 0.00 -> 10.6 mm
- net Net-(Q403B-B2): track 0.00 -> 10.5 mm
- net I2C5V_SCL_PROTEC: track 6.63 -> 16.5 mm
- net Net-(Q407B-B2): track 0.00 -> 9.65 mm
- net EPS_RESET: track 0.00 -> 9.52 mm
- net I2C33V_SCL: track 0.00 -> 9.43 mm
- net I2C5V_SDA: track 0.00 -> 9.41 mm
- net I2C33V_SDA: track 0.00 -> 8.96 mm
- net I2C5V_SCL: track 2.20 -> 8.97 mm
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Other:
- copper layers 2 -> 4
