File: One-U/One-U.kicad_pcb (KiCad board)
At the start: 2 copper layers, 96 x 89.9 mm, 107 parts, among them J1 SOLAR, J2 SOLAR, J3 SOLAR, J4 SOLAR, J5 SOLAR, SW1 SW_Push, U1 ATSAMD21J17A-M, U11 TMP117xxDRV, U12 TMP117xxDRV, U2 SPV1040TTR, U3 SPV1040TTR, U4 SPV1040TTR, U5 SPV1040TTR, U6 SPV1040TTR, U7 BNO055, Y1 Crystal_32.768kHz

Commit message: primitive one u
Parts:
- removed C_out10, C_out6, C_out8: 4.7uF, Capacitor_SMD:C_0603_1608Metric
- removed the C_out2 at (32.4, 32.9)
- removed the C_out4 at (36.4, 17.8)
- removed D1, D2, D3, D4, D5: D_Zener, Diode_SMD:D_1210_3225Metric
- removed H1: PC104-2*20, easyeda2kicad:HDR-TH_40P-P2.54-V-F-R2-C20-S2.54-2
- removed REF**: PC104-Standard, anant:PC104-Standard
- added H2: ~, anant:PC104-Standard, F.Cu at (163.8, 114.8)
- added U13: RFM69W, RF_Module:HOPERF_RFM69HW, F.Cu at (185.2, 108.6)
- C22, C23, C24, C25, C26, C35, C36, C37, C38, C39: footprint Capacitor_SMD:C_0805_2012Metric -> Capacitor_SMD:C_0603_1608Metric
- R21, R22, R23, R24: footprint Resistor_SMD:R_0805_2012Metric -> Resistor_SMD:R_0603_1608Metric
- Y1: footprint Crystal:Crystal_AT310_D3.0mm_L10.0mm_Horizontal -> Crystal:Crystal_AT310_D3.0mm_L10.0mm_Vertical
- moved L1 233.9 mm to (233.4, 53.1), turned to -90 degrees
- moved L2 228.2 mm to (233.4, 64.0), turned to -90 degrees
- moved R30 225.4 mm to (197.5, 115.6), turned to 180 degrees
- moved R27 225.2 mm to (195.2, 114.8), turned to -90 degrees
- moved L3 223.4 mm to (233.4, 75.2), turned to -90 degrees
- moved U2 220.6 mm to (224.9, 54.8), turned to 90 degrees
- moved L4 219.1 mm to (233.3, 86.2), turned to -90 degrees
- moved U3 218.6 mm to (224.9, 65.7), turned to 90 degrees
- moved U4 217.2 mm to (224.9, 76.9), turned to 90 degrees
- moved U5 216.3 mm to (224.8, 87.8), turned to 90 degrees
- moved U6 216.2 mm to (224.8, 99.1), turned to 90 degrees
- moved L5 215.8 mm to (233.3, 97.4), turned to -90 degrees
- moved C_IN5 215.2 mm to (235.5, 101.7)
- moved C20 213.4 mm to (229.5, 101.7)
- moved C_IN4 212.5 mm to (235.5, 90.5)
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- renumbered C_out3 to C_out2, C_out5 to C_out3, C_out7 to C_out4, C_out9 to C_out5
Connections:
- C22 pad 2: +3.3V -> VOUT_3.3V
- C40 pad 2: +3.3V -> VOUT_3.3V
- C41 pad 2: +3.3V -> VOUT_3.3V
- C_IN4 pad 1: INPUT5 -> INPUT4
- C_out1 pad 1: V_BUS_5V -> VIN
- C_out2 pad 1: V_BUS_5V -> VIN
- C_out3 pad 1: V_BUS_5V -> VIN
- C_out4 pad 1: V_BUS_5V -> VIN
- C_out5 pad 1: V_BUS_5V -> VIN
- L4 pad 2: INPUT5 -> INPUT4
- R10 pad 2: V_BUS_5V -> VIN
- R12 pad 1: INPUT5 -> INPUT4
- R13 pad 2: V_BUS_5V -> VIN
- R16 pad 2: V_BUS_5V -> VIN
- R18 pad 1: +3.3V -> VOUT_3.3V
- R19 pad 1: +3.3V -> VOUT_3.3V
- R27 pad 2: +3.3V -> VOUT_3.3V
- R30 pad 2: +3.3V -> VOUT_3.3V
- R4 pad 2: V_BUS_5V -> VIN
- R7 pad 2: V_BUS_5V -> VIN
- U1 pad 13: unconnected-(U1-PA04-Pad13) -> MISO
- U1 pad 14: unconnected-(U1-PA05-Pad14) -> CSLora
- U1 pad 15: unconnected-(U1-PA06-Pad15) -> MOSI
- U1 pad 16: unconnected-(U1-PA07-Pad16) -> SCK
- U1 pad 29: unconnected-(U1-PA12-Pad29) -> /SDA_3v
- U1 pad 30: unconnected-(U1-PA13-Pad30) -> /SCL_3v
- U1 pad 5: unconnected-(U1-PB04-Pad5) -> EN_5V
- U1 pad 6: unconnected-(U1-PB05-Pad6) -> EN_3.3V
- U1 pad 61: unconnected-(U1-PB00-Pad61) -> /TMP_MCU_INT1
- U1 pad 62: unconnected-(U1-PB01-Pad62) -> /TMP_MCU_INT2
- U1 pad 63: unconnected-(U1-PB02-Pad63) -> /BNO_INT3v
- U11 pad 5: +3.3V -> VOUT_3.3V
- U12 pad 4: +3.3V -> VOUT_3.3V
- U12 pad 5: +3.3V -> VOUT_3.3V
- U7 pad 14: /INT3v -> /BNO_INT3v
- U7 pad 28: +3.3V -> VOUT_3.3V
- U7 pad 3: +3.3V -> VOUT_3.3V
- U7 pad 4: +3.3V -> VOUT_3.3V
Routing:
- net INPUT5: track 0.00 -> 148.2 mm
- net INPUT4: track 0.00 -> 137.2 mm
- net INPUT3: track 0.00 -> 126.2 mm
- net INPUT2: track 0.00 -> 115.1 mm
- net INPUT1: track 0.00 -> 106.1 mm
- net VIN: track 0.00 -> 94.3 mm
- net VOUT_5V: track 0.00 -> 91.0 mm
- net /TMP_MCU_INT2: track 0.00 -> 89.3 mm, vias 0 -> 2
- net /SDA_3v: track 0.00 -> 86.0 mm, vias 0 -> 2
- net /SCL_3v: track 0.00 -> 83.7 mm, vias 0 -> 3
- net /TMP_MCU_INT1: track 0.00 -> 78.2 mm, vias 0 -> 2
- net EN_3.3V: track 0.00 -> 66.3 mm, vias 0 -> 2
- net EN_5V: track 0.00 -> 55.7 mm, vias 0 -> 2
- net /BNO_INT3v: track 0.00 -> 53.3 mm, vias 0 -> 2
- net MISO: track 0.00 -> 36.9 mm, vias 0 -> 2
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- added copper zone on In2.Cu, net GND
- added copper zone on In1.Cu, net VOUT_3.3V
Other:
- copper layers 2 -> 4

Commit message: more stuff on one u
Parts:
- added C34: 4.7uF, Capacitor_SMD:C_0603_1608Metric, F.Cu at (223.4, 115.2)
- added C42: 22uF, Capacitor_SMD:C_0603_1608Metric, F.Cu at (222.8, 105.8)
- added C43: 22uF, Capacitor_SMD:C_0603_1608Metric, F.Cu at (222.8, 104.0)
- added C44: 10uF, Capacitor_SMD:C_0603_1608Metric, F.Cu at (236.3, 110.1)
- added C45: 47uF, Capacitor_SMD:C_0603_1608Metric, F.Cu at (226.4, 113.8)
- added C46: 10uF, Capacitor_SMD:C_0603_1608Metric, F.Cu at (229.4, 113.8)
- added C47: 1uF, Capacitor_SMD:C_0603_1608Metric, F.Cu at (227.9, 109.4)
- added D3: LED, LED_SMD:LED_0603_1608Metric, F.Cu at (216.1, 115.9)
- added J8: Conn_01x02_Socket, Connector_AMASS:AMASS_XT30UPB-F_1x02_P5.0mm_Vertical, F.Cu at (247.2, 110.2)
- added J9: Conn_Coaxial_Small, Connector_Coaxial:SMA_Amphenol_132134-11_Vertical, F.Cu at (198.3, 102.6)
- added R32: 5.23k, Resistor_SMD:R_0603_1608Metric, F.Cu at (226.4, 116.8)
- added R33: 30.1k, Resistor_SMD:R_0603_1608Metric, F.Cu at (220.4, 116.7)
- added R34: 3.16k, Resistor_SMD:R_0603_1608Metric, F.Cu at (226.4, 115.2)
- added R35: 10k, Resistor_SMD:R_0603_1608Metric, F.Cu at (223.4, 116.7)
- added R36: 10k, Resistor_SMD:R_0603_1608Metric, F.Cu at (220.4, 115.2)
- added U8: BQ25883RGER, easyeda2kicad:VFQFPN-24_L4.0-W4.0-P0.50-BL-EP2.8, F.Cu at (222.0, 111.0)
- Y1: footprint Crystal:Crystal_AT310_D3.0mm_L10.0mm_Vertical -> Crystal:Crystal_AT310_D3.0mm_L10.0mm_Horizontal
- moved C10 1.95 mm to (183.3, 78.0)
- moved C11 1.95 mm to (183.3, 79.5)
- moved Y1 0.10 mm to (175.9, 72.7)
Connections:
- U1 pad 10: unconnected-(U1-PB07-Pad10) -> RST_TTC
- U1 pad 9: unconnected-(U1-PB06-Pad9) -> STAT
- U13 pad 10: unconnected-(U13-ANA-Pad10) -> Net-(J9-In)
Routing:
- net STAT: track 0.00 -> 58.9 mm, vias 0 -> 3
- net RST_TTC: track 0.00 -> 44.1 mm, vias 0 -> 2
- net VIN: track 94.3 -> 136.4 mm, vias 0 -> 2
- net V_BAT: track 0.00 -> 19.4 mm
- net Net-(C45-Pad2): track 0.00 -> 15.8 mm, vias 0 -> 2
- net /SCL_3v: track 83.7 -> 98.9 mm, vias 3 -> 4
- net /SDA_3v: track 86.0 -> 98.3 mm
- net THM: track 0.00 -> 10.0 mm
- net Net-(J9-In): track 0.00 -> 9.78 mm
- net Net-(U8-REGN): track 0.00 -> 5.79 mm, vias 0 -> 2
- net Net-(U8-ILIM): track 0.00 -> 5.60 mm
- net Net-(D3-A): track 0.00 -> 3.51 mm
- net Net-(U8-BTST): track 0.00 -> 2.66 mm
- net VOUT_5V: track 91.0 -> 93.4 mm
- net Net-(C34-Pad1): track 0.00 -> 1.52 mm
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