File: One-U/One-U.kicad_sch (KiCad schematic)
At the start: 115 parts, among them J1 SOLAR, J2 SOLAR, J3 SOLAR, J4 SOLAR, J5 SOLAR, SW1 SW_Push, U1 ATSAMD21J17A-M, U11 TMP117xxDRV, U12 TMP117xxDRV, U2 SPV1040TTR, U3 SPV1040TTR, U4 SPV1040TTR, U5 SPV1040TTR, U6 SPV1040TTR, U7 BNO055, U8 LTC2986HLX#PBF, Y1 Crystal_32.768kHz

Commit message: primitive one u
Parts:
- removed C27, C28, C29, C31: 10uF, Capacitor_SMD:C_0805_2012Metric, symbol Device:C
- removed C30: 0.1uF, Capacitor_SMD:C_0805_2012Metric, symbol Device:C
- removed C32, C34: 1uF, Capacitor_SMD:C_0805_2012Metric, symbol Device:C
- removed C33: 47uF, Capacitor_SMD:C_0805_2012Metric, symbol Device:C
- removed C_out10, C_out4, C_out6, C_out8: 4.7uF, Capacitor_SMD:C_0603_1608Metric, symbol Device:C
- removed D2, D3, D4, D5: D_Zener, Diode_SMD:D_1210_3225Metric, symbol Device:D_Zener
- removed H1: PC104-2*20, easyeda2kicad:HDR-TH_40P-P2.54-V-F-R2-C20-S2.54-2, symbol easyeda2kicad:PC104-2*20
- removed U8: LTC2986HLX#PBF, easyeda2kicad:LQFP-48_L7.0-W7.0-P0.50-LS9.0-BL, symbol easyeda2kicad:LTC2986HLX#PBF
- added H2: ~, anant:PC104-Standard, symbol ProjectLib:PC104
- added U13: RFM69W, RF_Module:HOPERF_RFM69HW, symbol RF_Module:RFM69W
- C22, C23, C24, C25, C26, C35, C36, C37, C38, C39: footprint Capacitor_SMD:C_0805_2012Metric -> Capacitor_SMD:C_0603_1608Metric
- C_outnn1: renamed from C_out2; now not fitted
- D1: now not fitted
- R21, R22, R23, R24: footprint Resistor_SMD:R_0805_2012Metric -> Resistor_SMD:R_0603_1608Metric
- Y1: footprint Crystal:Crystal_AT310_D3.0mm_L10.0mm_Horizontal -> Crystal:Crystal_AT310_D3.0mm_L10.0mm_Vertical
- renumbered C_out3 to C_out2, C_out5 to C_out3, C_out7 to C_out4, C_out9 to C_out5
Connections:
- net INT3v is gone; now on net BNO_INT3v: U7.14 (INT)
- net VOUT_3.3V is gone; now on net +3.3V: C38.1, C39.1, L8.2, R23.1
- net V_BUS_5V is gone; now on net VIN: C_out1.1, C_out2.1, C_out3.1, C_out4.1, C_out5.1, R10.2, R13.2, R16.2, R4.2, R7.2
- net +3.3V: now also H2.3, H2.39, U13.8 (3.3V)
- net EN_3.3V: now also U1.6 (PB05), H2.23
- net EN_5V: now also U1.5 (PB04), H2.25
- net GND: now also H2.1, U13.11 (GND), U13.9 (GND)
- net INPUT1: now also H2.43
- net INPUT2: now also H2.45
- net INPUT3: now also H2.47
- net INPUT4: now also C_IN4.1, L4.2, R12.1, H2.49
- net INPUT5: now also H2.51; no longer C_IN4.1, L4.2, R12.1
- net MISO: now also U1.13 (PA04), H2.9, U13.13 (MISO)
- net MOSI: now also U1.15 (PA06), H2.11, U13.14 (MOSI)
- net SCK: now also U1.16 (PA07), H2.7, U13.12 (SCK)
- net SCL_3v: now also U1.30 (PA13), H2.31
- net SDA_3v: now also U1.29 (PA12), H2.29
- net TMP_MCU_INT1: now also U1.61 (PB00), H2.8
- net TMP_MCU_INT2: now also U1.62 (PB01), H2.6
- net CSLora: now reaches U1.14 (PA05)
- net CSLora: now also H2.13, U13.15 (NSS)
- net BNO_INT3v: now reaches U1.63 (PB02)
- net BNO_INT3v: now also H2.32
- net VOUT_5V renamed +5V
- net +5V: now also H2.41, H2.5
- new net RST_TTC: U13.1 (RESET)
Other:
- note added: "LORA: RFM69W"
- note added: "Lora RADIO Module"
- note added: "NOTE: Switch from Connector instead of IC"
- note added: "SPV"
- note removed: "1. RESET PIN and CS PIN are ACTIVE LOW 2. INTERRUPT pin here is an outpin which gives LOW when the conversion cycle in the process and HIGH on the conclusion"
- note removed: "LTC2986"
- company: (none) -> Anant EPS
- title: (none) -> EPS ONE U PCB 
- moved on the sheet: C22, C23, C24, C25, C26, C35, C36, C37, C38, C39, L7, L8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

Commit message: more stuff on one u
Parts:
- added C27: 1uF, Capacitor_SMD:C_0603_1608Metric, symbol Device:C_Small
- added C28: 4.7uF, Capacitor_SMD:C_0603_1608Metric, symbol Device:C_Small
- added C29, C33: 10uF, Capacitor_SMD:C_0603_1608Metric, symbol Device:C_Small
- added C30: 47nF, Capacitor_SMD:C_0603_1608Metric, symbol Device:C_Small
- added C31, C32: 22uF, Capacitor_SMD:C_0603_1608Metric, symbol Device:C_Small
- added C34: 4.7uF, Capacitor_SMD:C_0603_1608Metric, symbol Device:C
- added C42, C43: 22uF, Capacitor_SMD:C_0603_1608Metric, symbol Device:C
- added C44, C46: 10uF, Capacitor_SMD:C_0603_1608Metric, symbol Device:C
- added C45: 47uF, Capacitor_SMD:C_0603_1608Metric, symbol Device:C
- added C47: 1uF, Capacitor_SMD:C_0603_1608Metric, symbol Device:C
- added D2: GREEN LED, LED_SMD:LED_0603_1608Metric, symbol Device:LED
- added D3: LED, LED_SMD:LED_0603_1608Metric, symbol Device:LED
- added J6: USB_C_Receptacle_USB2.0_16P, Connector_USB:USB_C_Receptacle_G-Switch_GT-USB-7010ASV, symbol Connector:USB_C_Receptacle_USB2.0_16P
- added J7: Conn_01x06, Connector_PinHeader_2.54mm:PinHeader_1x06_P2.54mm_Vertical, symbol Connector_Generic:Conn_01x06
- added J8: Conn_01x02_Socket, Connector_AMASS:AMASS_XT30UPB-F_1x02_P5.0mm_Vertical, symbol Connector:Conn_01x02_Socket
- added J9: Conn_Coaxial_Small, Connector_Coaxial:SMA_Amphenol_132134-11_Vertical, symbol Connector:Conn_Coaxial_Small
- added L9: 1uH, mainboard:L_2510, symbol Device:L
- added R25: 5.23K, Resistor_SMD:R_0603_1608Metric, symbol Device:R_US
- added R26: 30.1K, Resistor_SMD:R_0603_1608Metric, symbol Device:R_US
- added R28, R31: 10K, Resistor_SMD:R_0603_1608Metric, symbol Device:R_US
- added R29: 3.16K, Resistor_SMD:R_0603_1608Metric, symbol Device:R_US
- added R32: 5.23k, Resistor_SMD:R_0603_1608Metric, symbol Device:R
- added R33: 30.1k, Resistor_SMD:R_0603_1608Metric, symbol Device:R
- added R34: 3.16k, Resistor_SMD:R_0603_1608Metric, symbol Device:R
- added R35, R36: 10k, Resistor_SMD:R_0603_1608Metric, symbol Device:R
- added U14: BQ25883RGER, mainboard:QFN50P400X400X100-25N-D, symbol mainboard:BQ25883RGER
- added U8: BQ25883RGER, easyeda2kicad:VFQFPN-24_L4.0-W4.0-P0.50-BL-EP2.8, symbol easyeda2kicad:BQ25883RGER
- Y1: footprint Crystal:Crystal_AT310_D3.0mm_L10.0mm_Vertical -> Crystal:Crystal_AT310_D3.0mm_L10.0mm_Horizontal
Connections:
- net GND: now also C27.1, C29.1, C33.1, C42.2, C43.2, C44.1, C46.1, C47.1, J6.A1 (GND), J6.A12 (GND), J6.B1 (GND), J6.B12 (GND), J6.S1 (SHIELD), J7.5 (Pin_5), J7.6 (Pin_6), J8.1 (Pin_1), R33.2, R34.1, U14.19 (GND_1), U14.20 (GND_2), U14.25 (EP), U8.19 (GND), U8.20 (GND), U8.25 (EP)
- net RST_TTC: now also U1.10 (PB07)
- net SCL_3v: now also U8.5 (SCL)
- net SDA_3v: now also U8.4 (SDA)
- net VIN: now also C42.1, C43.1, C47.2, R32.1, U8.15 (SYS), U8.16 (SYS), U8.23 (VBUS)
- net at U13.10 (ANA): now also J9.1 (In)
- net STAT: now reaches U1.9 (PB06)
- net STAT: now also D2.1 (K), D3.1 (K), U14.2 (STAT), U8.2 (STAT)
- new net: C31.2, C32.2, J7.1 (Pin_1), U14.15 (SYS_1), U14.16 (SYS_2)
- new net: C34.1, R35.1
- new net: C33.2, J7.3 (Pin_3), U14.13 (BAT_1), U14.14 (BAT_2)
- new net: C34.2, R36.2, U8.11 (REGN)
- new net: C45.1, U8.12 (BTST)
- new net: C45.2, C46.2, U8.17 (SW), U8.18 (SW), U8.21 (PMID), U8.22 (PMID)
- new net: R34.2, U8.8 (ILIM)
- new net: R29.2, U14.8 (ILIM)
- new net: D2.2 (A), R31.1
- new net: C30.2, U14.12 (BTST)
- new net: C30.1, L9.2, U14.17 (SW_1), U14.18 (SW_2)
- new net: C29.2, L9.1, U14.21 (PMID_1), U14.22 (PMID_2)
- new net: D3.2 (A), R36.1
- new net GNDREF: C28.2, C31.1, C32.1, R26.1, R28.1, R29.1
- new net REGN: C28.1, R31.2, U14.11 (REGN)
- new net SCL_PWR: U14.5 (SCL)
- new net SDA_PWR: U14.4 (SDA)
- new net THM: R25.2, R26.2, R28.2, R32.2, R33.1, R35.2, U14.7 (TS), U8.7 (TS)
- new net USB_D+: J6.A6 (D+), J6.B6 (D+), U14.24 (D+)
- new net USB_D-: J6.A7 (D-), J6.B7 (D-), U14.1 (D-)
- new net VBATT: J7.2 (Pin_2)
- new net VBUS_IN: C27.2, J6.A4 (VBUS), J6.A9 (VBUS), J6.B4 (VBUS), J6.B9 (VBUS), R25.1, U14.23 (VBUS)
- new net VCHRG: J7.4 (Pin_4)
- new net V_BAT: C44.2, J8.2 (Pin_2), U8.13 (BAT), U8.14 (BAT)
- no-connect marks 0 -> 12
Other:
- note added: ""GND""
- note added: ""VCHRG""
- note added: ""VUSB""
- note added: "Add jumper to allow USB battery charging (even inside P-Pod)."
- note added: "Add jumper to allow USB to power the board (even inside P-Pod)."
- note added: "GARBAGE PART REMOVE AND ADD TO THE BUS"
- note added: "Input Current Limit Max input current (IINMAX)=KILIM/RILIM KILIM = 1098 to 1276 at most IINMAX=400mA=3.16 kohm"
- note added: "NOTE: Check what to do here ( sys to bus or what?)"
- note added: "RBF Jumpers"
- note added: "Remove both jumpers before flight to remove risk of unknown BQ25883 radiation failure modes"
- note added: "USB (Boost) Charging for 2-cell Li-Ion"
